File: BM83.kicad_sch (KiCad schematic)
At the start: 2 parts, among them IC1 BM83SM1-00AB, U1 Microchip_BM83

Commit message: ADC,充電管理IC，DCDC，CH32記載
Parts:
- removed IC1: BM83SM1-00AB, BM83SM100AA, symbol SamacSys_Parts:BM83SM1-00AB
- added C10, C4, C6, C8: 10u, symbol Device:C_Polarized_Small
- added C11, C12: 2.2u, symbol Device:C_Small
- added C13, C3: 2.2n, symbol Device:C_Small
- added C14: 10u, symbol Device:C_Small
- added C15, C16, C17, C2, C5, C7, C9: 0.1u, symbol Device:C_Small
- added D1: LED_Small, symbol Device:LED_Small
- added F1: Polyfuse, symbol Device:Polyfuse
- added FB1: 120, symbol Device:FerriteBead_Small
- added J1: Li-ion, symbol Connector_Generic:Conn_01x02
- added J24: USB_C_Receptacle_USB2.0, Connector_USB:USB_C_Receptacle_HRO_TYPE-C-31-M-12, symbol Connector:USB_C_Receptacle_USB2.0
- added JP1: UART/Write, symbol Jumper:Jumper_3_Bridged12
- added R1, R6: 10k, symbol Device:R_Small
- added R2, R3: 470, symbol Device:R_Small
- added R35, R36: 5.1k, Resistor_SMD:R_0603_1608Metric, symbol Device:R
- added R4, R5: 2k, symbol Device:R_Small
- added SW1: PowerON, symbol Switch:SW_SPST
- added U2: PCM5102A, Package_SO:TSSOP-20_4.4x6.5mm_P0.65mm, symbol Audio:PCM5102A
- added U3: CH32V003JxMx, Package_SO:JEITA_SOIC-8_3.9x4.9mm_P1.27mm, symbol MCU_WCH_RiscV:CH32V003JxMx
- added U4: MCP73831-2-OT, Package_TO_SOT_SMD:SOT-23-5, symbol Battery_Management:MCP73831-2-OT
- added U5: AE-XC9306-3V3, symbol My_Library:AE-XC9306-3V3
Connections:
- net AIR: now reaches U1.11 (AIR)
- net AIL: now reaches U1.12 (AIL)
- net GNDD: now reaches U1.16 (GND), U1.50 (GND), U1.56 (GND), U1.57 (GND)
- net GNDD: now also C14.2, C15.2, C16.2, C17.2, C2.2, C4.2, C5.1, C6.2, J1.2 (Pin_2), J24.A1 (GND), J24.A12 (GND), J24.B1 (GND), J24.B12 (GND), R4.2, SW1.1 (A), U2.10 (DEMP), U2.11 (FLT), U2.12 (SCK), U2.16 (FMT), U2.19 (DGND), U3.2 (VSS), U4.2 (V_{SS}), U5.2 (GND), U5.5 (GND)
- net LRCK: now reaches U1.2 (RFS1)
- net LRCK: now also U2.15 (LRCK)
- net +5V: now reaches U1.22 (ADAP_IN)
- net +5V: now also C17.1, D1.2 (A), F1.1, U4.4 (V_{DD})
- net +3.3V: now reaches U1.23 (BAT_IN)
- net +3.3V: now also C15.1, C16.1, C2.1, C4.1, FB1.1, R1.1, R6.1, U2.20 (DVDD), U3.4 (VDD), U5.3 (OUT)
- net at U1.26 (PWR(MFB)): now also R6.2, SW1.2 (B)
- net UART_TX_CH32: now reaches U1.29 (P8_6/UART_RXD)
- net UART_TX_CH32: now also JP1.1 (A)
- net BCK: now reaches U1.3 (SCLK1)
- net BCK: now also U2.13 (BCK)
- net UART_RX_CH32: now reaches U1.30 (P8_5/UART_TXD)
- net UART_RX_CH32: now also U3.1 (PD6/PA1)
- net LED1: now reaches U1.32 (LED1)
- net play/pause: now reaches U1.33 (P0_2)
- net LED2: now reaches U1.34 (LED2)
- net DM: now reaches U1.36 (DM)
- net DM: now also J24.A7 (D-), J24.B7 (D-)
- net DP: now reaches U1.37 (DP)
- net DP: now also J24.A6 (D+), J24.B6 (D+)
- net reverse: now reaches U1.38 (P0_3)
- net volume_up: now reaches U1.39 (P2_7)
- net DIN: now reaches U1.4 (DT1)
- net DIN: now also U2.14 (DIN)
- net volume_down: now reaches U1.40 (P0_5)
- net ~{RST}: now reaches U1.43 (~{RST})
- net foward: now reaches U1.44 (P0_1)
- net external codec reset: now reaches U1.49 (P0_0/UART_TX_IND)
- new net: D1.1 (K), R5.1
- new net: R5.2, U4.1 (STAT)
- new net: J24.B5 (CC2), R36.1
- new net: F1.2, J24.A4 (VBUS), J24.A9 (VBUS), J24.B4 (VBUS), J24.B9 (VBUS)
- new net: R3.2, U2.7 (OUTR)
- new net: J24.A5 (CC1), R35.1
- new net: JP1.2 (C), U3.8 (PD1/PD4/PD5)
- new net: R4.1, U4.5 (PROG)
- new net: R2.1, U2.6 (OUTL)
- new net: R1.2, U2.17 (XSMT)
- new net: C12.1, U2.2 (CAPP)
- new net: C12.2, U2.4 (CAPM)
- new net +3.3VA: C10.1, C7.1, C8.1, C9.1, FB1.2, U2.1 (CPVDD), U2.8 (AVDD)
- new net +BATT: C14.1, J1.1 (Pin_1), U4.3 (V_{BAT}), U5.1 (IN)
- new net AGND: C10.2, C11.1, C13.1, C3.2, C7.2, C8.2, C9.2, U2.3 (CPGND), U2.9 (AGND)
- new net AUDIO_L: C13.2, R2.2
- new net AUDIO_R: C3.1, R3.1
- new net GND: R35.2, R36.2
- new net LDOO: C5.2, C6.1, U2.18 (LDOO)
- new net SCL: U3.6 (PC2)
- new net SDA: U3.5 (PC1)
- new net SWIO: JP1.3 (B)
- new net VNEG: C11.2, U2.5 (VNEG)
- no-connect marks 0 -> 23
Other:
- note added: "BM83モジュールの設定について"
- note added: "Li-ion:1000mAh"
- note added: "OLEDこれ？"

Commit message: 回路図更新
Parts:
- added FB2: ?, symbol Device:FerriteBead_Small
- FB1: value 120 -> ?
- U4: value MCP73831-2-OT -> MCP73831
Connections:
- net AGND: now also FB2.2
- net GNDD: now also FB2.1
Other:
- moved on the sheet: C14, J1

Commit message: 回路図更新，昇圧どうしようね
Parts:
- added C1, C18: 470u, Capacitor_THT:CP_Radial_D16.0mm_P7.50mm, symbol Device:C_Polarized
- added C19: 0.1u, Capacitor_THT:C_Disc_D5.1mm_W3.2mm_P5.00mm, symbol Device:C
- added C20, C21: 0.1u, symbol Device:C
- added D2, D3, D4, D5: 1N4148, symbol Device:D_Small
- added D6: LED, LED_THT:LED_D3.0mm_Horizontal_O1.27mm_Z2.0mm, symbol Device:LED
- added D7, D8: D, Diode_THT:D_DO-35_SOD27_P7.62mm_Horizontal, symbol Device:D
- added NT1: NetTie_2, symbol Device:NetTie_2
- added Q1: 2SC1815, Package_TO_SOT_THT:TO-92L_Inline_Wide, symbol Simulation_SPICE:NPN
- added Q10, Q14: TTA004B, Package_TO_SOT_THT:TO-92L_Inline_Wide, symbol Transistor_BJT:Q_PNP_ECB
- added Q11, Q9: TTC004B, Package_TO_SOT_THT:TO-92L_Inline_Wide, symbol Transistor_BJT:Q_NPN_ECB
- added Q12, Q4, Q6, Q7: NPN, Package_TO_SOT_THT:TO-92L_Inline_Wide, symbol Transistor_BJT:Q_NPN_ECB
- added Q13, Q3, Q5, Q8: PNP, Package_TO_SOT_THT:TO-92L_Inline_Wide, symbol Transistor_BJT:Q_PNP_ECB
- added Q2: 2SA1015, Package_TO_SOT_THT:TO-92L_Inline_Wide, symbol Simulation_SPICE:PNP
- added R10, R7, R8, R9: 1k, symbol Device:R_Small
- added R11: 2k, Resistor_THT:R_Axial_DIN0204_L3.6mm_D1.6mm_P5.08mm_Horizontal, symbol Device:R
- added R12, R13: 10k, Resistor_THT:R_Axial_DIN0204_L3.6mm_D1.6mm_P5.08mm_Horizontal, symbol Device:R
- added R14: 220, Resistor_THT:R_Axial_DIN0204_L3.6mm_D1.6mm_P5.08mm_Horizontal, symbol Device:R
- added U6: Opamp_Dual, Package_DIP:DIP-8_W7.62mm_Socket, symbol Device:Opamp_Dual
Connections:
- net AGND: now also NT1.1
- net AUDIO_L: now also Q3.3 (B), Q4.3 (B)
- net AUDIO_R: now also Q5.3 (B), Q6.3 (B)
- new net: D3.1 (K), Q10.3 (B), R8.1
- new net: Q10.2 (C), R8.2
- new net: D5.1 (K), Q14.3 (B), R10.1
- new net: Q14.2 (C), R10.2
- new net: D2.1 (K), Q3.1 (E), Q7.3 (B)
- new net: D2.2 (A), Q9.3 (B), R7.2
- new net: Q7.1 (E), Q8.1 (E)
- new net: Q4.2 (C), Q7.2 (C), Q9.1 (E)
- new net: D5.2 (A), Q13.3 (B), Q6.1 (E)
- new net: Q11.1 (E), Q12.2 (C), Q6.2 (C)
- new net: R14.1, U6.1
- new net: Q1.2 (B), Q2.2 (B), R14.2
- new net: Q9.2 (C), R7.1
- new net: D6.1 (K), R11.1
- new net: R12.2, R13.1, U6.3 (+)
- new net: Q10.1 (E), Q3.2 (C), Q8.2 (C)
- new net: D3.2 (A), Q4.1 (E), Q8.3 (B)
- new net: D4.1 (K), Q12.3 (B), Q5.1 (E)
- new net: D4.2 (A), Q11.3 (B), R9.2
- new net: Q11.2 (C), R9.1
- new net: Q13.2 (C), Q14.1 (E), Q5.2 (C)
- new net: Q12.1 (E), Q13.1 (E)
- new net +12V: C1.1, C19.1, C20.1, D6.2 (A), D7.1 (K), Q1.1 (C), R12.1, U6.8 (V+)
- new net GNDREF: C1.2, C18.1, C20.2, C21.1, D7.2 (A), D8.1 (K), NT1.2, Q1.3 (E), Q2.3 (E), U6.2 (-)
- new net V_{-}: C18.2, C19.2, C21.2, D8.2 (A), Q2.1 (C), R11.2, R13.2, U6.4 (V-)
Other:
- note added: "HA-RZ710 105db/mW Z=48Ω PCM5102A Output voltage:2.1[VRMS]"
- note added: "heatsink"
- note added: "わかりやすかった"
- moved on the sheet: C10, C11, C15, C2, C4, C5, C6, C7, C8, C9, FB1

Commit message: 構成仮決定，sch内に記載
Other:
- note added: "・BM83→PCM5102A ・ライン入力 ・USB入力？ これらの後段でシングルエンド→差動変換 ・電圧増幅段:OPAMP ・出力段:ダイヤモンドバッファ ・電源20V ACアダプタ 数値要件は手元の紙参照"
Changed lines of the file:
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@@
 	(generator_version "10.0")
 	(paper "A4")
+	(text "・BM83→PCM5102A\n・ライン入力\n・USB入力？\nこれらの後段でシングルエンド→差動変換\n・電圧増幅段:OPAMP\n・出力段:ダイヤモンドバッファ\n・電源20V ACアダプタ\n\n数値要件は手元の紙参照"
+		(exclude_from_sim no)
+		(at 243.586 29.972 0)
+		(effects
+			(font
+				(size 1.27 1.27)
+			)
+			(justify left)
+		)
+	)
 	(text "heatsink"
 		(exclude_from_sim no)

Commit message: 回路図更新
Parts:
- removed C14: 10u, symbol Device:C_Small
- removed C15, C16, C17: 0.1u, symbol Device:C_Small
- removed D1: LED_Small, symbol Device:LED_Small
- removed FB1: ?, symbol Device:FerriteBead_Small
- removed J1: Li-ion, symbol Connector_Generic:Conn_01x02
- removed JP1: UART/Write, symbol Jumper:Jumper_3_Bridged12
- removed R4, R5: 2k, symbol Device:R_Small
- removed U3: CH32V003JxMx, Package_SO:JEITA_SOIC-8_3.9x4.9mm_P1.27mm, symbol MCU_WCH_RiscV:CH32V003JxMx
- removed U4: MCP73831, Package_TO_SOT_SMD:SOT-23-5, symbol Battery_Management:MCP73831-2-OT
- removed U5: AE-XC9306-3V3, symbol My_Library:AE-XC9306-3V3
- added C22: 0.1u, symbol Device:C
- added D1: D_Small, symbol Device:D_Small
- added FB3: ?, symbol Device:FerriteBead_Small
- added J1: Jack-DC, symbol Connector:Jack-DC
- added J2: AudioJack3, symbol Connector_Audio:AudioJack3
- added SW2: SW_Slide_DPDT, symbol Switch:SW_Slide_DPDT
- added U3: STM32G431KBTx, Package_QFP:LQFP-32_7x7mm_P0.8mm, symbol MCU_ST_STM32G4:STM32G431KBTx
- added U4: USBLC6-2SC6, Package_TO_SOT_SMD:SOT-23-6, symbol Power_Protection:USBLC6-2SC6
Connections:
- net GND is gone; now on net GNDD: R35.2, R36.2
- net +5V: now also D1.1 (K); no longer F1.1
- net DM: now also SW2.2 (B), U4.6 (I/O1); no longer J24.A7 (D-), J24.B7 (D-)
- net DP: now also SW2.5 (B), U4.4 (I/O2); no longer J24.A6 (D+), J24.B6 (D+)
- net GNDD: now also C22.2, J1.2, U4.2 (GND)
- net at F1.2, J24.A4 (VBUS), J24.A9 (VBUS)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: now also U4.5 (VBUS)
- net +12V renamed VDD
- net VDD: now also C22.1, FB3.2
- net UART_RX_CH32 renamed UART_RX_STM
- net UART_TX_CH32 renamed UART_TX_STM
- new net: D1.2 (A), F1.1
- new net: U3.16 (VSS), U3.32 (VSS)
- new net: J24.A6 (D+), J24.B6 (D+), U4.3 (I/O2)
- new net: J24.A7 (D-), J24.B7 (D-), U4.1 (I/O1)
- new net: FB3.1, J1.1
- new net SWCLK: SW2.6 (C)
- new net SWDIO: SW2.1 (A)
- new net USB_DM: SW2.3 (C)
- new net USB_DP: SW2.4 (A)
- no-connect marks 23 -> 19
Other:
- note added: "PMOS+PTCサーミスタでポップノイズ対策？"
- note added: "VDD->DCDC->5V VDD->DCDC->3.3VD->filter->3.3VA"
- note added: "双二次フィルタの話"
- note removed: "Li-ion:1000mAh"
- moved on the sheet: F1, R35, R36

Commit message: 差動変換とか書いた
Parts:
- removed D2, D3, D4, D5: 1N4148, symbol Device:D_Small
- removed Q10, Q14: TTA004B, Package_TO_SOT_THT:TO-92L_Inline_Wide, symbol Transistor_BJT:Q_PNP_ECB
- removed Q11, Q9: TTC004B, Package_TO_SOT_THT:TO-92L_Inline_Wide, symbol Transistor_BJT:Q_NPN_ECB
- removed Q12, Q4, Q6, Q7: NPN, Package_TO_SOT_THT:TO-92L_Inline_Wide, symbol Transistor_BJT:Q_NPN_ECB
- removed Q13, Q3, Q5, Q8: PNP, Package_TO_SOT_THT:TO-92L_Inline_Wide, symbol Transistor_BJT:Q_PNP_ECB
- removed R10, R7, R8, R9: 1k, symbol Device:R_Small
- removed SW2: SW_Slide_DPDT, symbol Switch:SW_Slide_DPDT
- added C14, C15: 0.22u, Capacitor_THT:C_Rect_L7.2mm_W3.5mm_P5.00mm, symbol Device:C
- added C16, C17: 1u, Capacitor_THT:C_Rect_L7.2mm_W6.0mm_P5.00mm, symbol Device:C
- added C23, C24: 0.022u, Capacitor_THT:C_Rect_L7.2mm_W2.5mm_P5.00mm, symbol Device:C
- added C25, C26: 0.1u, Capacitor_THT:C_Rect_L7.2mm_W2.5mm_P5.00mm, symbol Device:C
- added C27, C28: 2200p, Capacitor_THT:C_Rect_L7.2mm_W2.5mm_P5.00mm, symbol Device:C
- added C29, C30: 0.01u, Capacitor_THT:C_Rect_L7.2mm_W2.5mm_P5.00mm, symbol Device:C
- added C31, C32, C33, C34: 4.7u, symbol Device:C_Small
- added C35: 0.33u, symbol Device:C_Small
- added C36: 2.2u, symbol Device:C_Small
- added IC1: NJM2845DL1-33, TO-252-3-L1, symbol SamacSys_Parts:NJM2845DL1-33-TE1
- added JP1, JP2: Jumper_3_Open, symbol Jumper:Jumper_3_Open
- added L1, L2: 3.3u, symbol Device:L_Small
- added PS1: M78AR05-0.5, M78AR03305, symbol SamacSys_Parts:M78AR05-0.5
- added PS2: M78AR033-0.5, M78AR03305, symbol SamacSys_Parts:M78AR033-0.5
- added Q15, Q18: PNP, Package_TO_SOT_THT:TO-92L_Inline_Wide, symbol Transistor_BJT:Q_PNP_ECB
- added Q16, Q17: NPN, Package_TO_SOT_THT:TO-92L_Inline_Wide, symbol Transistor_BJT:Q_NPN_ECB
- added R10, R15, R18, R19, R22, R23: 47k, Resistor_THT:R_Axial_DIN0204_L3.6mm_D1.6mm_P5.08mm_Horizontal, symbol Device:R
- added R16, R17, R20, R21, R8, R9: 680, Resistor_THT:R_Axial_DIN0204_L3.6mm_D1.6mm_P5.08mm_Horizontal, symbol Device:R
- added R24, R25, R42, R43, R44, R45, R46, R47, R48, R49, R5, R50, R51, R52, R53, R7: 10k, Resistor_THT:R_Axial_DIN0204_L3.6mm_D1.6mm_P5.08mm_Horizontal, symbol Device:R
- added R27, R28: 1k, Resistor_THT:R_Axial_DIN0204_L3.6mm_D1.6mm_P5.08mm_Horizontal, symbol Device:R
- added R31, R32: 2.2, Resistor_THT:R_Axial_DIN0207_L6.3mm_D2.5mm_P7.62mm_Horizontal, symbol Device:R
- added R37, R38: 100k, Resistor_THT:R_Axial_DIN0204_L3.6mm_D1.6mm_P5.08mm_Horizontal, symbol Device:R_Small
- added RV1, RV2, RV3, RV4, RV5: 10k, MyLibrary:SL4515G, symbol MysymbolLibrary:RV_2C
- added U10, U11: Opamp_Quad, symbol Device:Opamp_Quad
- added U5: TL072, Package_DIP:DIP-8_W7.62mm_Socket, symbol Device:Opamp_Dual
- added U7, U8: TL074, Package_DIP:DIP-14_W7.62mm_Socket, symbol Device:Opamp_Quad
- added U9: Opamp_Dual, symbol Device:Opamp_Dual
Connections:
- net AUDIO_L is gone; now on net SIG_L: C13.2, R2.2
- net AUDIO_R is gone; now on net SIG_R: C3.1, R3.1
- net +3.3V: now also C36.1, IC1.3 (VOUT); no longer U1.23 (BAT_IN)
- net +3.3VA: now also PS2.3 (VOUT)
- net +5V: now also C33.1, C35.1, IC1.1 (VIN), L2.1, PS1.3 (VOUT)
- net AGND: now also C33.2, C34.2, PS2.2 (GND)
- net DM: now also JP2.2 (C)
- net DP: now also JP1.2 (C)
- net GNDD: now also U3.14 (VSSA), U3.16 (VSS), U3.32 (VSS), C31.2, C32.2, C35.2, C36.2, IC1.2 (GND), PS1.2 (GND)
- net GNDREF: now also J2.S, R10.2, R15.2, R18.2, R19.2, R22.2, R23.2, R37.2, R38.2, R45.2, R47.2, R50.2, R51.2, RV4.3, RV5.3, U10.3 (+), U11.3 (+)
- net SWCLK: now also JP1.1 (A)
- net SWDIO: now also JP2.1 (A)
- net USB_DM: now also JP2.3 (B)
- net USB_DP: now also JP1.3 (B)
- net VDD: now also C32.1, L1.1, Q16.2 (C), Q17.2 (C), R27.1
- net V_{-}: now also Q15.2 (C), Q18.2 (C), R28.2
- net SIG_R: now reaches J2.R
- net SIG_R: now also R38.1, U5.5 (+)
- net SIG_L: now reaches J2.T
- net SIG_L: now also R37.1, U5.3 (+)
- new net: Q16.1 (E), Q18.3 (B), R28.1
- new net: C14.1, RV1.2
- new net: C14.2, C16.1, R8.1
- new net: R43.1, RV4.2, U10.5 (+)
- new net: R46.1, R47.1, U10.6 (-)
- new net: R49.2, U11.1, U11.10 (+)
- new net: R48.2, R49.1, U11.2 (-)
- new net: R51.1, R53.1, U11.9 (-)
- new net: R8.2, U7.1, U7.2 (-)
- new net: C27.2, C29.1, R20.1
- new net: C29.2, R22.1, U7.12 (+)
- new net: R48.1, RV5.2, U11.5 (+)
- new net: C31.1, L1.2, PS1.1 (VIN)
- new net: Q15.1 (E), Q17.3 (B), R27.2
- new net: R50.1, R52.1, U11.6 (-)
- new net: C28.2, C30.1, R21.1
- new net: C30.2, R23.1, U8.10 (+)
- new net: C24.1, RV2.5
- new net: C24.2, C26.1, R17.1
- new net: C34.1, L2.2, PS2.1 (VIN)
- new net: R5.1, U5.1, U5.2 (-)
- new net: C26.2, R19.1, U8.5 (+)
- new net: R17.2, U8.6 (-), U8.7
- new net: C23.2, C25.1, R16.1
- new net: C25.2, R18.1, U7.5 (+)
- new net: R44.1, R45.1, U10.9 (-)
- new net: R25.1, RV1.4, RV2.4, RV3.4, U8.13 (-)
- new net: R7.2, RV1.6, RV2.6, RV3.6, U8.12 (+)
- new net: R24.1, RV1.1, RV2.1, RV3.1, U7.9 (-)
- new net: R5.2, RV1.3, RV2.3, RV3.3, U7.10 (+)
- new net: R42.2, U10.1, U10.10 (+)
- new net: R16.2, U7.6 (-), U7.7
- new net: Q17.1 (E), R31.1
- new net: R31.2, R32.1
- new net: C16.2, R10.1, U7.3 (+)
- new net: C27.1, RV3.2
- new net: Q18.1 (E), R32.2
- new net: R20.2, U7.13 (-), U7.14
- new net: R21.2, U8.8, U8.9 (-)
- new net: C28.1, RV3.5
- new net: C17.2, R15.1, U8.3 (+)
- new net: C15.1, RV1.5
- new net: C23.1, RV2.2
- new net: R7.1, U5.6 (-), U5.7
- new net: C15.2, C17.1, R9.1
- new net: R42.1, R43.2, U10.2 (-)
- new net: R9.2, U8.1, U8.2 (-)
- new net COLD: R44.2, R53.2, U10.8, U11.8
- new net EQ_L: R24.2, RV4.1, U7.8
- new net EQ_R: R25.2, RV5.1, U8.14
- new net HOT: R46.2, R52.2, U10.7, U11.7
- no-connect marks 19 -> 20
Other:
- note added: "100Hz"
- note added: "10kHz"
- note added: "1kHz"
- note added: "Equalizer"
- note added: "Ra"
- note added: "Ra=Rb, A=(Rc+Rd)/Rd"
- note added: "Rb"
- note added: "Rc"
- note added: "Rd"
- note added: "STM32G431KB"
- note added: "シングルエンド‐差動変換 増幅段"
- note added: "バッファ"
- note added: "ライン入力"
- note added: "・BM83→PCM5102A ・ライン入力 ・USB入力？ これらの後段でシングルエンド→差動変換 ・電圧増幅段:OPAMP ・出力段:ダイヤモンドバッファ ・電源24V ACアダプタ 数値要件は手元の紙参照"
- note added: "出力段"
- note added: "定電流回路とかの話"
- note added: "書き込み/接続用USB"
- note added: "電源"
- note removed: "VDD->DCDC->5V VDD->DCDC->3.3VD->filter->3.3VA"
- note removed: "heatsink"
- note removed: "わかりやすかった"
- note removed: "・BM83→PCM5102A ・ライン入力 ・USB入力？ これらの後段でシングルエンド→差動変換 ・電圧増幅段:OPAMP ・出力段:ダイヤモンドバッファ ・電源20V ACアダプタ 数値要件は手元の紙参照"
- moved on the sheet: C22, FB3, J1, J2

Commit message: 回路図ほぼ書いて整えた
Parts:
- removed C1, C18: 470u, Capacitor_THT:CP_Radial_D16.0mm_P7.50mm, symbol Device:C_Polarized
- removed C10, C4, C6, C8: 10u, symbol Device:C_Polarized_Small
- removed C11, C12, C36: 2.2u, symbol Device:C_Small
- removed C13, C3: 2.2n, symbol Device:C_Small
- removed C14, C15: 0.22u, Capacitor_THT:C_Rect_L7.2mm_W3.5mm_P5.00mm, symbol Device:C
- removed C16, C17: 1u, Capacitor_THT:C_Rect_L7.2mm_W6.0mm_P5.00mm, symbol Device:C
- removed C19: 0.1u, Capacitor_THT:C_Disc_D5.1mm_W3.2mm_P5.00mm, symbol Device:C
- removed C2, C5, C7, C9: 0.1u, symbol Device:C_Small
- removed C20, C21: 0.1u, symbol Device:C
- removed C23, C24: 0.022u, Capacitor_THT:C_Rect_L7.2mm_W2.5mm_P5.00mm, symbol Device:C
- removed C25, C26: 0.1u, Capacitor_THT:C_Rect_L7.2mm_W2.5mm_P5.00mm, symbol Device:C
- removed C27, C28: 2200p, Capacitor_THT:C_Rect_L7.2mm_W2.5mm_P5.00mm, symbol Device:C
- removed C29, C30: 0.01u, Capacitor_THT:C_Rect_L7.2mm_W2.5mm_P5.00mm, symbol Device:C
- removed C31, C32, C33, C34: 4.7u, symbol Device:C_Small
- removed C35: 0.33u, symbol Device:C_Small
- removed D6: LED, LED_THT:LED_D3.0mm_Horizontal_O1.27mm_Z2.0mm, symbol Device:LED
- removed D7, D8: D, Diode_THT:D_DO-35_SOD27_P7.62mm_Horizontal, symbol Device:D
- removed IC1: NJM2845DL1-33, TO-252-3-L1, symbol SamacSys_Parts:NJM2845DL1-33-TE1
- removed L1, L2: 3.3u, symbol Device:L_Small
- removed PS1: M78AR05-0.5, M78AR03305, symbol SamacSys_Parts:M78AR05-0.5
- removed PS2: M78AR033-0.5, M78AR03305, symbol SamacSys_Parts:M78AR033-0.5
- removed Q1: 2SC1815, Package_TO_SOT_THT:TO-92L_Inline_Wide, symbol Simulation_SPICE:NPN
- removed Q15, Q18: PNP, Package_TO_SOT_THT:TO-92L_Inline_Wide, symbol Transistor_BJT:Q_PNP_ECB
- removed Q16, Q17: NPN, Package_TO_SOT_THT:TO-92L_Inline_Wide, symbol Transistor_BJT:Q_NPN_ECB
- removed Q2: 2SA1015, Package_TO_SOT_THT:TO-92L_Inline_Wide, symbol Simulation_SPICE:PNP
- removed R1, R6: 10k, symbol Device:R_Small
- removed R10, R15, R18, R19, R22, R23: 47k, Resistor_THT:R_Axial_DIN0204_L3.6mm_D1.6mm_P5.08mm_Horizontal, symbol Device:R
- removed R11: 2k, Resistor_THT:R_Axial_DIN0204_L3.6mm_D1.6mm_P5.08mm_Horizontal, symbol Device:R
- removed R12, R13, R24, R25, R42, R43, R44, R45, R46, R47, R48, R49, R5, R50, R51, R52, R53, R7: 10k, Resistor_THT:R_Axial_DIN0204_L3.6mm_D1.6mm_P5.08mm_Horizontal, symbol Device:R
- removed R14: 220, Resistor_THT:R_Axial_DIN0204_L3.6mm_D1.6mm_P5.08mm_Horizontal, symbol Device:R
- removed R16, R17, R20, R21, R8, R9: 680, Resistor_THT:R_Axial_DIN0204_L3.6mm_D1.6mm_P5.08mm_Horizontal, symbol Device:R
- removed R2, R3: 470, symbol Device:R_Small
- removed R27, R28: 1k, Resistor_THT:R_Axial_DIN0204_L3.6mm_D1.6mm_P5.08mm_Horizontal, symbol Device:R
- removed R31, R32: 2.2, Resistor_THT:R_Axial_DIN0207_L6.3mm_D2.5mm_P7.62mm_Horizontal, symbol Device:R
- removed R35, R36: 5.1k, Resistor_SMD:R_0603_1608Metric, symbol Device:R
- removed RV1, RV2, RV3, RV4, RV5: 10k, MyLibrary:SL4515G, symbol MysymbolLibrary:RV_2C
- removed SW1: PowerON, symbol Switch:SW_SPST
- removed U1: Microchip_BM83, RF_Module:Microchip_BM83, symbol RF_Bluetooth:Microchip_BM83
- removed U10, U11: Opamp_Quad, symbol Device:Opamp_Quad
- removed U2: PCM5102A, Package_SO:TSSOP-20_4.4x6.5mm_P0.65mm, symbol Audio:PCM5102A
- removed U3: STM32G431KBTx, Package_QFP:LQFP-32_7x7mm_P0.8mm, symbol MCU_ST_STM32G4:STM32G431KBTx
- removed U5: TL072, Package_DIP:DIP-8_W7.62mm_Socket, symbol Device:Opamp_Dual
- removed U6: Opamp_Dual, Package_DIP:DIP-8_W7.62mm_Socket, symbol Device:Opamp_Dual
- removed U7, U8: TL074, Package_DIP:DIP-14_W7.62mm_Socket, symbol Device:Opamp_Quad
- removed U9: Opamp_Dual, symbol Device:Opamp_Dual
- added C102, C103: 0.1u, symbol Device:C_Small
- added D102: ?, symbol Device:D_Zener
- added D103, D104, D105, D106, D107: LED, symbol Device:LED_Small
- added FB101: 60, symbol Device:FerriteBead_Small
- added H101, H102, H103, H104: M3, symbol Mechanical:MountingHole_Pad
- added J104, J105: Conn_01x02, symbol Connector_Generic:Conn_01x02
- added NT101: NetTie_2, symbol Device:NetTie_2
- added R103, R104, R106, R107, R108, R109, R110, R111: 10k, symbol Device:R_Small
- added R105: 47k, symbol Device:R_Small
- added SW101: SW_Slide_DPDT, symbol Switch:SW_Slide_DPDT
- added U102: CH221K, Package_TO_SOT_SMD:SOT-23-6, symbol Interface_USB:CH221K
- D101: renamed from D1; value D_Small -> ?
- renumbered C22 to C101, F1 to F101, FB3 to FB102, FB2 to FB103, J1 to J101, J2 to J102, J24 to J103, JP1 to JP101, JP2 to JP102, NT1 to NT102, R37 to R101, R38 to R102, U4 to U101
Connections:
- net +3.3V: now also D106.2 (A)
- net +3.3VA: now also D107.2 (A)
- net +5V: now also D105.2 (A); no longer D101.1 (K)
- net AGND: now also R111.2
- net GNDD: now also C102.1, C103.2, D102.2 (A), FB101.2, NT101.2, R103.2, R104.2, R109.2, R110.2, U102.2 (GND); no longer C101.2, J101.2
- net GNDREF: now also H101.1, H102.1, H103.1, H104.1
- net USB_DM: now also SW101.2 (B)
- net USB_DP: now also SW101.5 (B)
- net VDD: now also D104.2 (A); no longer C101.1, FB102.2
- net at J103.B5 (CC2): now also R103.1, U102.5 (CC2)
- net at D101.2 (A), F101.1: now also C102.2, D102.1 (K), R105.1
- net at J103.A5 (CC1): now also R104.1, U102.4 (CC1)
- net at J103.S1 (SHIELD): now also FB101.1
- new net: D103.1 (K), R108.1
- new net: D104.1 (K), R107.1
- new net: C103.1, R105.2, R106.1, U102.1 (VDD)
- new net: R106.2, U102.6 (CFG)
- new net: D106.1 (K), R110.1
- new net: D107.1 (K), R111.1
- new net: D105.1 (K), R109.1
- new net Amplifier/OUT_L+: J104.1 (Pin_1)
- new net Amplifier/OUT_L-: J104.2 (Pin_2)
- new net Amplifier/OUT_R+: J105.1 (Pin_1)
- new net Amplifier/OUT_R-: J105.2 (Pin_2)
- new net DM_BM83: SW101.3 (C)
- new net DM_STM32: SW101.1 (A)
- new net DP_BM83: SW101.4 (A)
- new net DP_STM32: SW101.6 (C)
- new net GNDPWR: C101.2, J101.2, NT101.1, R107.2, R108.2
- new net VIN: C101.1, D101.1 (K), D103.2 (A), FB102.2
- no-connect marks 20 -> 3
Other:
- added sheet Amplifier (Amplifier.kicad_sch)
- added sheet DAC (DAC.kicad_sch)
- added sheet Equalizer (Equalizer.kicad_sch)
- added sheet Power (Power.kicad_sch)
- note added: "ST7735S接続参考"
- note added: "インバーテッドダーリントン"
- note added: "ダイヤモンドバッファ"
- note added: "ダーリントン接続"
- note added: "・BM83→PCM5102A ・ライン入力 ・USB入力？ これらの後段でシングルエンド→差動変換 ・電圧増幅段:OPAMP ・出力段:ダイヤモンドバッファ ・電源12V ACアダプタ & UPB PD 12V(差動である点に留意) ・電源優先回路(ACアダプタ優先) 数値要件は手元の紙参照"
- note added: "書き込み/UAC接続/給電用USB"
- note removed: "100Hz"
- note removed: "10kHz"
- note removed: "1kHz"
- note removed: "Equalizer"
- note removed: "PMOS+PTCサーミスタでポップノイズ対策？"
- note removed: "Ra"
- note removed: "Ra=Rb, A=(Rc+Rd)/Rd"
- note removed: "Rb"
- note removed: "Rc"
- note removed: "Rd"
- note removed: "STM32G431KB"
- note removed: "シングルエンド‐差動変換 増幅段"
- note removed: "バッファ"
- note removed: "ライン入力"
- note removed: "・BM83→PCM5102A ・ライン入力 ・USB入力？ これらの後段でシングルエンド→差動変換 ・電圧増幅段:OPAMP ・出力段:ダイヤモンドバッファ ・電源24V ACアダプタ 数値要件は手元の紙参照"
- note removed: "出力段"
- note removed: "書き込み/接続用USB"
- note removed: "電源"
- moved on the sheet: C101, D101, F101, FB102, FB103, J101, J102, J103, JP101, JP102, NT102, R101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
