File: BM83.kicad_sch (KiCad schematic)
At the start: 76 parts, among them IC101 NJM2845DL1-33, J101 USB_C_Receptacle_USB2.0, J102 Conn_01x02, J103 Jack-DC, J104 3557-2, J105 Conn_01x02, J106 AudioJack3, K101 DG85B-7011-75-1024, Q101 2SC1815, Q102 2SA1015, SW101 SW_Slide_DPDT, SW102 SW_SPST, U101 CH221K, U102 USBLC6-2SC6, U103 LM358N

Commit message: 部品ほぼ割り当て
Parts:
- removed FB101: ?, symbol Device:FerriteBead_Small
- removed NT101, NT102: NetTie_2, symbol Device:NetTie_2
- added C119, C120: 1u, Capacitor_THT:C_Rect_L7.2mm_W6.0mm_P5.00mm, symbol Device:C_Small
- C101, C102, C103, C108, C111, C113, C114: footprint (none) -> Capacitor_SMD:C_1206_3216Metric
- C104, C105, C106, C107: footprint Capacitor_THT:CP_Radial_D16.0mm_P7.50mm -> Capacitor_THT:CP_Radial_D12.5mm_P5.00mm
- C110: footprint Capacitor_THT:C_Disc_D5.1mm_W3.2mm_P5.00mm -> Capacitor_SMD:C_0603_1608Metric
- C115, C116, C117, C118: footprint (none) -> Capacitor_SMD:C_0603_1608Metric
- D101, D102, D103, D104, D105: footprint (none) -> LED_THT:LED_D5.0mm_Horizontal_O1.27mm_Z3.0mm
- D106: footprint (none) -> nittc-footprint-library:CUHS20F30H3F
- D107: footprint (none) -> Diode_THT:D_DO-35_SOD27_P7.62mm_Horizontal
- D108: footprint samacsys:CUHS20F30H3F -> nittc-footprint-library:CUHS20F30H3F
- D109, D111: footprint Diode_THT:D_DO-35_SOD27_P7.62mm_Horizontal -> (none)
- F101: footprint (none) -> nittc-footprint-library:MFRX110720
- FB101: renamed from FB102; footprint (none) -> Inductor_SMD:L_0603_1608Metric
- FB102: renamed from FB103; footprint (none) -> Inductor_SMD:L_0603_1608Metric
- H101, H102, H103, H104: footprint (none) -> MountingHole:MountingHole_3.2mm_M3_Pad_Via
- IC101: footprint TO-252-3-L1 -> Package_TO_SOT_SMD:TO-252-2
- J102, J105: footprint (none) -> Connector_JST:JST_VH_B2P-VH_1x02_P3.96mm_Vertical
- J103: footprint (none) -> Connector_BarrelJack:BarrelJack_Horizontal
- J104: footprint samacsys:3557-2 -> nittc-footprint-library:fuse_holder
- J106: footprint (none) -> MyLibrary:MJ352W
- JP101, JP102: footprint (none) -> Connector_PinHeader_2.54mm:PinHeader_1x03_P2.54mm_Vertical
- K101: value DG85B-7011-75-1024 -> G2R-1-E 24V; footprint MyLibrary:DG85B-7011-75-1024 -> (none)
- L101, L102: footprint (none) -> MyLibrary:744774033
- PS101, PS102: footprint M78AR03305 -> MyLibrary:M78A
- R101, R102, R103, R104, R105: footprint (none) -> Resistor_SMD:R_0603_1608Metric
- R106: value 47k -> 1k; footprint (none) -> Resistor_SMD:R_2512_6332Metric
- R107: value 10k -> 200k; footprint (none) -> Resistor_SMD:R_0603_1608Metric
- R108, R109: value 10k -> 5.1k; footprint (none) -> Resistor_SMD:R_0603_1608Metric
- R110: footprint (none) -> MyLibrary:CEMENT_RESISTOR_5W
- R111, R112, R113, R114, R115, R116: footprint Resistor_THT:R_Axial_DIN0204_L3.6mm_D1.6mm_P5.08mm_Horizontal -> Resistor_SMD:R_0603_1608Metric
- SW101: footprint (none) -> Button_Switch_THT:SW_E-Switch_EG2219_DPDT_Angled
- SW102: footprint (none) -> Connector_JST:JST_XH_B2B-XH-A_1x02_P2.50mm_Vertical
Connections:
- net GNDD is gone; now on net AGND: C101.1, C102.2, C113.2, C114.2, C117.2, C118.2, D107.2 (A), FB101.2, IC101.2 (GND), J101.A1 (GND), J101.A12 (GND), J101.B1 (GND), J101.B12 (GND), PS101.2 (GND), R103.2, R104.2, R108.2, R109.2, U101.2 (GND), U102.2 (GND)
- net GNDPWR is gone; now on net AGND: C103.2, C104.2, C105.2, C106.2, C107.2, D108.2 (A), J103.2, K101.86 (COIL_2), R101.2, R102.2
- net AGND: now also J106.S
- net GNDREF: no longer J106.S
- net SIG_L: now also C119.2; no longer J106.T
- net SIG_R: now also C120.1; no longer J106.R
- new net: C120.2, J106.R
- new net: C119.1, J106.T
Other:
- note added: "1kR 6432 2W"
- note added: "DPDT"
- note added: "Polyfuse"
- note added: "SBD"
- note added: "TVS"
- note added: "インダクタ"
- note added: "リレー"
- moved on the sheet: J106

Commit message: 何やってたか忘れた
Parts:
- removed D110: LED, LED_THT:LED_D3.0mm_Horizontal_O1.27mm_Z2.0mm, symbol Device:LED
- removed R113: 2k, Resistor_SMD:R_0603_1608Metric, symbol Device:R
- removed U102: USBLC6-2SC6, Package_TO_SOT_SMD:SOT-23-6, symbol Power_Protection:USBLC6-2SC6
- added D108, D109: PESD5V0S1UL, Diode_SMD:D_SOD-882, symbol Device:D_Zener_Small
- C104, C105, C106, C107: footprint Capacitor_THT:CP_Radial_D12.5mm_P5.00mm -> Capacitor_THT:CP_Radial_D16.0mm_P7.50mm
- C110: footprint Capacitor_SMD:C_0603_1608Metric -> Capacitor_SMD:C_1206_3216Metric
- D101, D102, D103, D104, D105: footprint LED_THT:LED_D5.0mm_Horizontal_O1.27mm_Z3.0mm -> LED_THT:LED_D3.0mm_Horizontal_O1.27mm_Z2.0mm
- D107: value ? -> SMF24A; footprint Diode_THT:D_DO-35_SOD27_P7.62mm_Horizontal -> Diode_SMD:D_SOD-123F
- D111: renamed from D109; footprint (none) -> nittc-footprint-library:CUHS20F30H3F
- D112: renamed from D111; footprint (none) -> nittc-footprint-library:CUHS20F30H3F
- FB102: value ? -> 33; footprint Inductor_SMD:L_0603_1608Metric -> Inductor_SMD:L_0805_2012Metric
- J106: footprint MyLibrary:MJ352W -> samacsys:MJ-8435
- JP101, JP102: footprint Connector_PinHeader_2.54mm:PinHeader_1x03_P2.54mm_Vertical -> Jumper:SolderJumper-3_P1.3mm_Open_RoundedPad1.0x1.5mm
- K101: footprint (none) -> Relay_THT:Relay_SPDT_Omron_G2RL-1-E
- renumbered C119 to C117, C120 to C118, C117 to C119, C118 to C120, D108 to D110, R114 to R113, R115 to R114, R116 to R115, U103 to U102
Connections:
- net V- is gone; now on net AGND: C110.2, C111.2, C112.2, D112.2 (A), Q102.1 (C), R113.2, U102.4 (V-)
- net AGND: now also H101.1, H102.1, H103.1, H104.1, K101.A2 (COIL_2), D108.2 (A), D109.2 (A); no longer K101.86 (COIL_2)
- net DM: now also J101.A7 (D-), J101.B7 (D-), D108.1 (K)
- net DP: now also J101.A6 (D+), J101.B6 (D+), D109.1 (K)
- net DP_BM83: now also SW101.6 (A); no longer SW101.4 (A)
- net DP_STM32: now also SW101.4 (C); no longer SW101.6 (C)
- net GNDREF: no longer H101.1, H102.1, H103.1, H104.1
- net V+: now also K101.14 (NO); no longer K101.87 (NO)
- net at J104.2, J104.4, R110.1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: now also K101.11 (COM); no longer K101.30 (COM)
- net at D110.1 (K), SW102.2 (B): now also K101.A1 (COIL_1); no longer K101.85 (COIL_1)
- net USB_DM renamed USB_D-
- net USB_DP renamed USB_D+
Other:
- note added: "1000uF"
- note added: "TVS for DPDM"
- note added: "TVS for VBUS"
- note added: "フェライトビーズ"
- note removed: "TVS"
- moved on the sheet: C117, C118, J106, R114, R115

Commit message: 部品配置すすめた
Other:
- note added: "つまみ"
Changed lines of the file:
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@@
+		)
+	)
+	(text "つまみ"
+		(exclude_from_sim no)
+		(at 203.708 150.114 0)
+		(effects
+			(font
+				(size 1.27 1.27)
+			)
+			(href "https://akizukidenshi.com/catalog/g/g112202/")
 		)
 	)

Commit message: 回路図一部変更，部品ほぼ置いた　寝かせる
Parts:
- added C121: 1000u, Capacitor_THT:CP_Radial_D16.0mm_P7.50mm, symbol Device:C_Polarized
- J102, J105: value Conn_01x02 -> JST_VH
Connections:
- net AGND: now also C121.2
- net V+: now also C121.1
Other:
- note added: "←@20V,4000uF"
Changed lines of the file:
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@@
 		)
 	)
+	(text "←@20V,4000uF"
+		(exclude_from_sim no)
+		(at 112.522 81.788 0)
+		(effects
+			(font
+				(size 1.27 1.27)
+			)
+		)
+	)
 	(text "双二次フィルタの話"
 		(exclude_from_sim no)
@@
 	)
 	(junction
+		(at 121.92 104.14)
+		(diameter 0)
+		(color 0 0 0 0)
+	)
+	(junction
 		(at 74.93 138.43)
 		(diameter 0)
@@
 	)
 	(junction
+		(at 128.27 93.98)
+		(diameter 0)
+		(color 0 0 0 0)
+	)
+	(junction
 		(at 40.64 53.34)
 		(diameter 0)
@@
 	(wire
 		(pts
+			(xy 128.27 102.87) (xy 128.27 104.14)
+		)
+		(stroke
+			(width 0)
+			(type default)
+		)
+	)
+	(wire
+		(pts
 			(xy 217.17 93.98) (xy 227.33 93.98)
 		)
@@
 	(wire
 		(pts
+			(xy 128.27 93.98) (xy 128.27 95.25)
+		)
+		(stroke
+			(width 0)
+			(type default)
+		)
+	)
+	(wire
+		(pts
 			(xy 50.8 152.4) (xy 50.8 153.67)
 		)
@@
 	(wire
 		(pts
+			(xy 121.92 104.14) (xy 128.27 104.14)
+		)
+		(stroke
+			(width 0)
+			(type default)
+		)
+	)
+	(wire
+		(pts
 			(xy 74.93 118.11) (xy 74.93 119.38)
 		)
@@
 	(wire
 		(pts
+			(xy 128.27 93.98) (xy 121.92 93.98)
+		)
+		(stroke
+			(width 0)
+			(type default)
+		)
+	)
+	(wire
+		(pts
 			(xy 39.37 132.08) (xy 39.37 135.89)
 		)
@@
 			)
 		)
-		(property "Value" "Conn_01x02"
+		(property "Value" "JST_VH"
 			(at 256.54 88.8999 0)
 			(show_name no)
@@
 	)
 	(symbol
+		(lib_id "Device:C_Polarized")
+		(at 128.27 99.06 0)
+		(unit 1)
+		(body_style 1)
+		(exclude_from_sim no)
+		(in_bom yes)
+		(on_board yes)
+		(in_pos_files yes)
+		(dnp no)
+		(property "Reference" "C121"
+			(at 128.27 106.172 0)
+			(show_name no)
+			(do_not_autoplace no)
+			(effects
+				(font
+					(size 1.27 1.27)
+				)
+				(justify left)
+			)
+		)
+		(property "Value" "1000u"
+			(at 128.27 108.712 0)
+			(show_name no)
+			(do_not_autoplace no)
+			(effects
+				(font
+					(size 1.27 1.27)
+				)
+				(justify left)
+			)
+		)
+		(property "Footprint" "Capacitor_THT:CP_Radial_D16.0mm_P7.50mm"
+			(at 129.2352 102.87 0)
+			(hide yes)
+			(show_name no)
+			(do_not_autoplace no)
+			(effects
+				(font
+					(size 1.27 1.27)
+				)
+			)
+		)
+		(property "Datasheet" ""
+			(at 128.27 99.06 0)
+			(hide yes)
+			(show_name no)
+			(do_not_autoplace no)
+			(effects
+				(font
+					(size 1.27 1.27)
+				)
+			)
+		)
+		(property "Description" "Polarized capacitor"
+			(at 128.27 99.06 0)
+			(hide yes)
+			(show_name no)
+			(do_not_autoplace no)
+			(effects
+				(font
+					(size 1.27 1.27)
+				)
+			)
+		)
+		(pin "2"
+		)
+		(pin "1"
+		)
+		(instances
+			(project "BM83"
+				(path "/00b28691-5113-4bf2-bf96-cb8ff43f915f"
+					(reference "C121")
+					(unit 1)
+				)
+			)
+		)
+	)
+	(symbol
 		(lib_id "power:VCC")
 		(at 101.6 118.11 0)
@@
 	(symbol
 		(lib_id "power:VDD")
-		(at 121.92 93.98 0)
+		(at 128.27 93.98 0)
 		(unit 1)
 		(body_style 1)
@@
 		(dnp no)
 		(property "Reference" "#PWR0124"
-			(at 121.92 97.79 0)
+			(at 128.27 97.79 0)
 			(hide yes)
 			(show_name no)
@@
 		)
 		(property "Value" "VDD"
-			(at 121.92 90.17 0)
+			(at 128.27 90.17 0)
 			(show_name no)
 			(do_not_autoplace no)
@@
 		)
 		(property "Footprint" ""
-			(at 121.92 93.98 0)
+			(at 128.27 93.98 0)
 			(hide yes)
 			(show_name no)
@@
 		)
 		(property "Datasheet" ""
-			(at 121.92 93.98 0)
+			(at 128.27 93.98 0)
 			(hide yes)
 			(show_name no)
@@
 		)
 		(property "Description" "Power symbol creates a global label with name \"VDD\""
-			(at 121.92 93.98 0)
+			(at 128.27 93.98 0)
 			(hide yes)
 			(show_name no)
@@
 			)
 		)
-		(property "Value" "Conn_01x02"
+		(property "Value" "JST_VH"
 			(at 256.54 99.0599 0)
 			(show_name no)

Commit message: 部品配置進行中
Connections:
- net DM_BM83 renamed BM83_D-
- net DM_STM32 renamed STM32_D-
- net DP_BM83 renamed BM83_D+
- net DP_STM32 renamed STM32_D+
Other:
- sheet DAC ports: added SWCLK, SWDIO; removed none
- note added: "↑接続先確認(AGNDではないか)"
Changed lines of the file:
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@@
 		)
 	)
+	(text "↑接続先確認(AGNDではないか)"
+		(exclude_from_sim no)
+		(at 268.478 61.468 0)
+		(effects
+			(font
+				(size 1.27 1.27)
+			)
+		)
+	)
 	(text "つまみ"
 		(exclude_from_sim no)
@@
 	(wire
 		(pts
+			(xy 165.1 81.28) (xy 168.91 81.28)
+		)
+		(stroke
+			(width 0)
+			(type default)
+		)
+	)
+	(wire
+		(pts
 			(xy 110.49 40.64) (xy 114.3 40.64)
 		)
@@
 	(wire
 		(pts
-			(xy 165.1 88.9) (xy 168.91 88.9)
+			(xy 165.1 93.98) (xy 168.91 93.98)
 		)
 		(stroke
@@
 	(wire
 		(pts
-			(xy 165.1 96.52) (xy 168.91 96.52)
+			(xy 165.1 101.6) (xy 168.91 101.6)
 		)
 		(stroke
@@
 	(wire
 		(pts
-			(xy 165.1 86.36) (xy 168.91 86.36)
+			(xy 165.1 91.44) (xy 168.91 91.44)
 		)
 		(stroke
@@
 	(wire
 		(pts
+			(xy 165.1 83.82) (xy 168.91 83.82)
+		)
+		(stroke
+			(width 0)
+			(type default)
+		)
+	)
+	(wire
+		(pts
 			(xy 26.67 172.72) (xy 26.67 173.99)
 		)
@@
 	(wire
 		(pts
-			(xy 165.1 99.06) (xy 168.91 99.06)
+			(xy 165.1 104.14) (xy 168.91 104.14)
 		)
 		(stroke
@@
 		)
 	)
-	(label "DP_BM83"
-		(at 165.1 96.52 180)
+	(label "SWCLK"
+		(at 165.1 81.28 180)
 		(effects
 			(font
@@
 		)
 	)
-	(label "DP_STM32"
-		(at 165.1 86.36 180)
+	(label "STM32_D-"
+		(at 165.1 93.98 180)
+		(effects
+			(font
+				(size 1.27 1.27)
+			)
+			(justify right bottom)
+		)
+	)
+	(label "STM32_D+"
+		(at 165.1 91.44 180)
 		(effects
 			(font
@@
 		)
 	)
+	(label "BM83_D-"
+		(at 165.1 104.14 180)
+		(effects
+			(font
+				(size 1.27 1.27)
+			)
+			(justify right bottom)
+		)
+	)
 	(label "USB_D+"
 		(at 119.38 67.31 0)
@@
 		)
 	)
-	(label "DM_BM83"
+	(label "BM83_D-"
 		(at 109.22 72.39 180)
 		(effects
@@
 		)
 	)
-	(label "DM_BM83"
-		(at 165.1 99.06 180)
+	(label "BM83_D+"
+		(at 119.38 72.39 0)
 		(effects
 			(font
 				(size 1.27 1.27)
 			)
-			(justify right bottom)
+			(justify left bottom)
 		)
 	)
-	(label "DP_BM83"
-		(at 119.38 72.39 0)
+	(label "SWDIO"
+		(at 165.1 83.82 180)
 		(effects
 			(font
 				(size 1.27 1.27)
 			)
-			(justify left bottom)
+			(justify right bottom)
 		)
 	)
-	(label "DM_STM32"
-		(at 165.1 88.9 180)
+	(label "BM83_D+"
+		(at 165.1 101.6 180)
 		(effects
 			(font
@@
 		)
 	)
-	(label "DP_STM32"
-		(at 119.38 62.23 0)
+	(label "STM32_D-"
+		(at 109.22 62.23 180)
 		(effects
 			(font
 				(size 1.27 1.27)
 			)
-			(justify left bottom)
+			(justify right bottom)
 		)
 	)
-	(label "DM_STM32"
-		(at 109.22 62.23 180)
+	(label "STM32_D+"
+		(at 119.38 62.23 0)
 		(effects
 			(font
 				(size 1.27 1.27)
 			)
-			(justify right bottom)
+			(justify left bottom)
 		)
 	)
@@
 	)
 	(sheet
-		(at 168.91 83.82)
-		(size 19.05 17.78)
+		(at 168.91 78.74)
+		(size 19.05 27.94)
 		(exclude_from_sim no)
 		(in_bom yes)
@@
 		)
 		(property "Sheetname" "DAC"
-			(at 168.91 83.1084 0)
+			(at 168.91 78.0284 0)
 			(show_name no)
 			(do_not_autoplace no)
@@
 		)
 		(property "Sheetfile" "DAC.kicad_sch"
-			(at 168.91 102.1846 0)
+			(at 168.91 107.2646 0)
 			(show_name no)
 			(do_not_autoplace no)
@@
 		)
 		(pin "DP_BM83" input
-			(at 168.91 96.52 180)
+			(at 168.91 101.6 180)
 			(effects
 				(font
@@
 		)
 		(pin "DM_STM" input
-			(at 168.91 88.9 180)
+			(at 168.91 93.98 180)
 			(effects
 				(font
@@
 		)
 		(pin "DP_STM" input
-			(at 168.91 86.36 180)
+			(at 168.91 91.44 180)
 			(effects
 				(font
@@
 		)
 		(pin "DM_BM83" input
-			(at 168.91 99.06 180)
+			(at 168.91 104.14 180)
+			(effects
+				(font
+					(size 1.27 1.27)
+				)
+				(justify left)
+			)
+		)
+		(pin "SWCLK" input
+			(at 168.91 81.28 180)
+			(effects
+				(font
+					(size 1.27 1.27)
+				)
+				(justify left)
+			)
+		)
+		(pin "SWDIO" bidirectional
+			(at 168.91 83.82 180)
 			(effects
 				(font

Commit message: Volumeの種類と位置変えた
Parts:
- C109, C112: footprint Capacitor_THT:CP_Radial_D16.0mm_P7.50mm -> Capacitor_THT:CP_Radial_D10.0mm_P5.00mm
Other:
- note added: "電解コンデンサ"
Changed lines of the file:
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@@
 		)
 	)
+	(text "電解コンデンサ"
+		(exclude_from_sim no)
+		(at 112.776 127.508 0)
+		(effects
+			(font
+				(size 1.27 1.27)
+			)
+			(href "https://akizukidenshi.com/catalog/g/g102719/")
+		)
+	)
 	(junction
 		(at 63.5 118.11)
@@
 			)
 		)
-		(property "Footprint" "Capacitor_THT:CP_Radial_D16.0mm_P7.50mm"
+		(property "Footprint" "Capacitor_THT:CP_Radial_D10.0mm_P5.00mm"
 			(at 91.1352 137.16 0)
 			(hide yes)
@@
 			)
 		)
-		(property "Footprint" "Capacitor_THT:CP_Radial_D16.0mm_P7.50mm"
+		(property "Footprint" "Capacitor_THT:CP_Radial_D10.0mm_P5.00mm"
 			(at 91.1352 127 0)
 			(hide yes)
