File: Power.kicad_sch (KiCad schematic)
At the start: 35 parts, among them IC401 NJM2845DL1-33, J401 3557-2, K401 DG85B-7011-75-1024, Q401 2SC1815, Q402 2SA1015, SW401 SW_SPST, U401 LM358N

Commit message: 回路図ひとまず完成
Parts:
- renumbered C407 to C406, C406 to C407
Changed lines of the file:
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@@
 		(dnp no)
 		(property "Reference" "C408"
-			(at 127.508 70.104 0)
+			(at 124.46 65.532 0)
 			(show_name no)
 			(do_not_autoplace no)
@@
 		)
 		(property "Value" "1000u"
-			(at 127.508 72.644 0)
+			(at 124.46 68.072 0)
 			(show_name no)
 			(do_not_autoplace no)
@@
 		(in_pos_files yes)
 		(dnp no)
-		(property "Reference" "C407"
+		(property "Reference" "C406"
 			(at 115.824 114.3 0)
 			(show_name no)
@@
 			(project "BM83"
 				(path "/00b28691-5113-4bf2-bf96-cb8ff43f915f/91566e44-dea6-486b-a621-3d20a30261fd"
-					(reference "C407")
+					(reference "C406")
 					(unit 1)
 				)
@@
 		(in_pos_files yes)
 		(dnp no)
-		(property "Reference" "C406"
-			(at 121.158 70.104 0)
+		(property "Reference" "C407"
+			(at 118.11 65.532 0)
 			(show_name no)
 			(do_not_autoplace no)
@@
 		)
 		(property "Value" "1000u"
-			(at 121.158 72.644 0)
+			(at 118.11 68.072 0)
 			(show_name no)
 			(do_not_autoplace no)
@@
 			(project "BM83"
 				(path "/00b28691-5113-4bf2-bf96-cb8ff43f915f/91566e44-dea6-486b-a621-3d20a30261fd"
-					(reference "C406")
+					(reference "C407")
 					(unit 1)
 				)
@@
 		(dnp no)
 		(property "Reference" "C410"
-			(at 140.208 70.104 0)
+			(at 137.16 65.532 0)
 			(show_name no)
 			(do_not_autoplace no)
@@
 		)
 		(property "Value" "1000u"
-			(at 140.208 72.644 0)
+			(at 137.16 68.072 0)
 			(show_name no)
 			(do_not_autoplace no)
@@
 		(dnp no)
 		(property "Reference" "C409"
-			(at 133.858 70.104 0)
+			(at 130.81 65.532 0)
 			(show_name no)
 			(do_not_autoplace no)
@@
 		)
 		(property "Value" "1000u"
-			(at 133.858 72.644 0)
-			(show_name no)
-			(do_not_autoplace no)
+			(at 130.81 68.072 0)
+			(show_name no)
+			(do_not_autoplace no)
