File: DAC.kicad_sch (KiCad schematic)
At the start: 33 parts, among them SW501 PowerON, SW502 SW_Push, U501 STM32G431KBTx, U502 Microchip_BM83, U503 ST7735S, U504 PCM5102A

Commit message: 回路図ひとまず完成
Parts:
- renumbered C508 to C201, C509 to C202, C507 to C203, C510 to C204, C515 to C205, C511 to C206, C516 to C207, C512 to C208, C517 to C209, C513 to C210, C514 to C211, C518 to C212, C501 to C213, C502 to C214, C503 to C215, C504 to C216, C505 to C217, C506 to C218, LED501 to LED201, LED502 to LED202, R503 to R201, R504 to R202, R502 to R203, R501 to R204, RV501 to RV201, RV502 to RV202, RV503 to RV203, SW501 to SW201, SW502 to SW202, U504 to U201, U502 to U202, U503 to U203, U501 to U204
Other:
- moved on the sheet: C204, C205, C206, C207, C208, C209, C210, C211, C212

Commit message: 部品ほぼ割り当て
Parts:
- removed RV201, RV202, RV203: 10k, symbol Device:R_Potentiometer
- added C219, C220: 1u, Capacitor_THT:C_Rect_L7.2mm_W6.0mm_P5.00mm, symbol Device:C_Small
- added R205, R206: 100k, Resistor_SMD:R_0603_1608Metric, symbol Device:R_Small
- added R207, R208, R209, R210, R211, R212: 10k, Resistor_SMD:R_0603_1608Metric, symbol Device:R
- added SW203, SW204, SW205, SW206, SW207, SW208: SW_Push, symbol Switch:SW_Push
- C201, C202, C203, C204, C206, C208, C210, C211, C213: footprint (none) -> Capacitor_SMD:C_0603_1608Metric
- C205, C207, C209, C212: footprint (none) -> Capacitor_SMD:CP_Elec_3x5.3
- LED201, LED202: footprint WS2812B:WS2812B-NARROW -> LED_SMD:LED_WS2812B_PLCC4_5.0x5.0mm_P3.2mm
- R201, R202, R203, R204: footprint (none) -> Resistor_SMD:R_0603_1608Metric
- SW201: footprint (none) -> Connector_JST:JST_XH_B2B-XH-A_1x02_P2.50mm_Vertical
- SW202: footprint (none) -> samacsys:TVAF06A020BR
- U203: footprint (none) -> Connector_JST:JST_XH_B8B-XH-A_1x08_P2.50mm_Vertical
Connections:
- net +3.3V: now also SW203.2, SW204.2, SW205.2, SW206.2, SW207.2, SW208.2
- net AGND: now also R205.1, R206.2
- net GNDD: now also R207.2, R208.2, R209.2, R210.2, R211.2, R212.2
- net SIG_L: now also C219.2, R205.2; no longer C201.2, R201.2
- net SIG_R: now also C220.1, R206.1; no longer C202.1, R202.1
- net PB3: now reaches U204.26 (PB3)
- net PB3: now also R207.1, SW203.1
- net PB4: now reaches U204.27 (PB4)
- net PB4: now also R208.1, SW204.1
- net PB5: now reaches U204.28 (PB5)
- net PB5: now also R209.1, SW205.1
- net PB6: now reaches U204.29 (PB6)
- net PB6: now also R210.1, SW206.1
- net PB7: now reaches U204.30 (PB7)
- net PB7: now also R211.1, SW207.1
- net PB8: now reaches U204.31 (PB8)
- net PB8: now also R212.1, SW208.1
- net ADC1_IN1: no longer names the net of U204.5 (PA0)
- net ADC1_IN2: no longer names the net of U204.6 (PA1)
- net ADC1_IN3: no longer names the net of U204.7 (PA2)
- new net: C202.1, C220.2, R202.1
- new net: C201.2, C219.1, R201.2
Other:
- note added: "10uF"
- note added: "2.2Vくらいだった気がする"
- note added: "タクトスイッチ縦"
- note added: "デジタルイコライザ"

Commit message: 何やってたか忘れた
Parts:
- removed C218: 0.1u, Capacitor_SMD:C_0603_1608Metric, symbol Device:C
- removed SW203, SW204, SW205, SW206, SW207, SW208: SW_Push, symbol Switch:SW_Push
- added SW202, SW203, SW204: TL53BF160Q, samacsys:TL53BF160Q, symbol MysymbolLibrary:TL53BF160Q
- C216: renamed from C214; footprint Capacitor_SMD:C_0603_1608Metric -> Capacitor_SMD:C_0402_1005Metric
- C217: renamed from C215; footprint Capacitor_SMD:C_0603_1608Metric -> Capacitor_SMD:C_0402_1005Metric
- C218: renamed from C216; footprint Capacitor_SMD:C_0603_1608Metric -> Capacitor_SMD:C_0402_1005Metric
- C219: renamed from C217; footprint Capacitor_SMD:C_0603_1608Metric -> Capacitor_SMD:C_0402_1005Metric
- renumbered C219 to C202, C220 to C203, C202 to C204, C203 to C205, C204 to C206, C205 to C207, C206 to C208, C207 to C209, C208 to C210, C209 to C211, C210 to C212, C211 to C213, C212 to C214, C213 to C215, R205 to R201, R201 to R202, R202 to R203, R206 to R204, R203 to R205, R204 to R206, R209 to R208, R211 to R209, R208 to R210, R210 to R211, SW202 to SW205
Connections:
- net +3.3V: now also SW202.3, SW202.4, SW203.3, SW203.4, SW204.3, SW204.4
- net PB3: now also SW202.1
- net PB4: now also SW202.2
- net PB5: now also SW203.1
- net PB6: now also SW203.2
- net PB7: now also SW204.1
- net PB8: now also SW204.2
- net RESET: now reaches C215.1, SW205.2, U204.4 (PG10)
- no-connect marks 19 -> 43
Other:
- note added: "タクトスイッチ縦2連"
- note removed: "タクトスイッチ縦"

Commit message: 部品配置すすめた
Parts:
- C201, C204, C205, C206, C208, C210, C212, C213: footprint Capacitor_SMD:C_0603_1608Metric -> Capacitor_SMD:C_0402_1005Metric
Connections:
- net VDD1 is gone; now on net +3.3V: C218.1, U204.1 (VDD)
- net VDD2 is gone; now on net +3.3V: C219.1, U204.17 (VDD)
- net VDDA is gone; now on net +3.3VA: C216.1, C217.1, U204.15 (VDDA)
Changed lines of the file:
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@@
 	(wire
 		(pts
+			(xy 59.69 123.19) (xy 66.04 123.19)
+		)
+		(stroke
+			(width 0)
+			(type default)
+		)
+	)
+	(wire
+		(pts
 			(xy 189.23 45.72) (xy 190.5 45.72)
 		)
@@
 	(wire
 		(pts
+			(xy 59.69 129.54) (xy 68.58 129.54)
+		)
+		(stroke
+			(width 0)
+			(type default)
+		)
+	)
+	(wire
+		(pts
 			(xy 273.05 128.27) (xy 273.05 129.54)
 		)
@@
 		)
 	)
+	(label "VDDA"
+		(at 66.04 123.19 90)
+		(effects
+			(font
+				(size 1.27 1.27)
+			)
+			(justify left bottom)
+		)
+	)
 	(label "foward"
 		(at 85.09 41.91 0)
@@
 		)
 	)
+	(label "VDD2"
+		(at 68.58 129.54 90)
+		(effects
+			(font
+				(size 1.27 1.27)
+			)
+			(justify left bottom)
+		)
+	)
 	(label "AIL"
 		(at 38.1 80.01 180)
@@
 		)
 	)
+	(label "VDD1"
+		(at 66.04 129.54 90)
+		(effects
+			(font
+				(size 1.27 1.27)
+			)
+			(justify left bottom)
+		)
+	)
 	(label "volume_down"
 		(at 85.09 49.53 0)
@@
 			)
 		)
-		(property "Footprint" "Capacitor_SMD:C_0603_1608Metric"
+		(property "Footprint" "Capacitor_SMD:C_0402_1005Metric"
 			(at 181.61 52.07 0)
 			(hide yes)
@@
 			)
 		)
-		(property "Footprint" "Capacitor_SMD:C_0603_1608Metric"
+		(property "Footprint" "Capacitor_SMD:C_0402_1005Metric"
 			(at 171.45 58.42 0)
 			(hide yes)
@@
 			)
 		)
-		(property "Footprint" "Capacitor_SMD:C_0603_1608Metric"
+		(property "Footprint" "Capacitor_SMD:C_0402_1005Metric"
 			(at 186.69 88.9 0)
 			(hide yes)
@@
 			)
 		)
-		(property "Footprint" "Capacitor_SMD:C_0603_1608Metric"
+		(property "Footprint" "Capacitor_SMD:C_0402_1005Metric"
 			(at 186.69 72.39 0)
 			(hide yes)
@@
 			)
 		)
-		(property "Footprint" "Capacitor_SMD:C_0603_1608Metric"
+		(property "Footprint" "Capacitor_SMD:C_0402_1005Metric"
 			(at 186.69 83.82 0)
 			(hide yes)
@@
 			)
 		)
-		(property "Footprint" "Capacitor_SMD:C_0603_1608Metric"
+		(property "Footprint" "Capacitor_SMD:C_0402_1005Metric"
 			(at 181.61 44.45 0)
 			(hide yes)
@@
 	)
 	(symbol
+		(lib_id "power:+3.3VA")
+		(at 59.69 123.19 0)
+		(unit 1)
+		(body_style 1)
+		(exclude_from_sim no)
+		(in_bom yes)
+		(on_board yes)
+		(in_pos_files yes)
+		(dnp no)
+		(property "Reference" "#PWR0232"
+			(at 59.69 127 0)
+			(hide yes)
+			(show_name no)
+			(do_not_autoplace no)
+			(effects
+				(font
+					(size 1.27 1.27)
+				)
+			)
+		)
+		(property "Value" "+3.3VA"
+			(at 59.69 119.38 0)
+			(show_name no)
+			(do_not_autoplace no)
+			(effects
+				(font
+					(size 1.27 1.27)
+				)
+			)
+		)
+		(property "Footprint" ""
+			(at 59.69 123.19 0)
+			(hide yes)
+			(show_name no)
+			(do_not_autoplace no)
+			(effects
+				(font
+					(size 1.27 1.27)
+				)
+			)
+		)
+		(property "Datasheet" ""
+			(at 59.69 123.19 0)
+			(hide yes)
+			(show_name no)
+			(do_not_autoplace no)
+			(effects
+				(font
+					(size 1.27 1.27)
+				)
+			)
+		)
+		(property "Description" "Power symbol creates a global label with name \"+3.3VA\""
+			(at 59.69 123.19 0)
+			(hide yes)
+			(show_name no)
+			(do_not_autoplace no)
+			(effects
+				(font
+					(size 1.27 1.27)
+				)
+			)
+		)
+		(pin "1"
+		)
+		(instances
+			(project "BM83"
+				(path "/00b28691-5113-4bf2-bf96-cb8ff43f915f/514f5709-5940-41c3-bb07-e91835a532d4"
+					(reference "#PWR0232")
+					(unit 1)
+				)
+			)
+		)
+	)
+	(symbol
 		(lib_id "WS2812B:WS2812B")
 		(at 167.64 154.94 0)
@@
 			)
 		)
-		(property "Footprint" "Capacitor_SMD:C_0603_1608Metric"
+		(property "Footprint" "Capacitor_SMD:C_0402_1005Metric"
 			(at 186.69 101.6 0)
 			(hide yes)
@@
 	)
 	(symbol
+		(lib_id "power:+3.3V")
+		(at 59.69 129.54 0)
+		(unit 1)
+		(body_style 1)
+		(exclude_from_sim no)
+		(in_bom yes)
+		(on_board yes)
+		(in_pos_files yes)
+		(dnp no)
+		(property "Reference" "#PWR0231"
+			(at 59.69 133.35 0)
+			(hide yes)
+			(show_name no)
+			(do_not_autoplace no)
+			(effects
+				(font
+					(size 1.27 1.27)
+				)
+			)
+		)
+		(property "Value" "+3.3V"
+			(at 59.69 125.73 0)
+			(show_name no)
+			(do_not_autoplace no)
+			(effects
+				(font
+					(size 1.27 1.27)
+				)
+			)
+		)
+		(property "Footprint" ""
+			(at 59.69 129.54 0)
+			(hide yes)
+			(show_name no)
+			(do_not_autoplace no)
+			(effects
+				(font
+					(size 1.27 1.27)
+				)
+			)
+		)
+		(property "Datasheet" ""
+			(at 59.69 129.54 0)
+			(hide yes)
+			(show_name no)
+			(do_not_autoplace no)
+			(effects
+				(font
+					(size 1.27 1.27)
+				)
+			)
+		)
+		(property "Description" "Power symbol creates a global label with name \"+3.3V\""
+			(at 59.69 129.54 0)
+			(hide yes)
+			(show_name no)
+			(do_not_autoplace no)
+			(effects
+				(font
+					(size 1.27 1.27)
+				)
+			)
+		)
+		(pin "1"
+		)
+		(instances
+			(project "BM83"
+				(path "/00b28691-5113-4bf2-bf96-cb8ff43f915f/514f5709-5940-41c3-bb07-e91835a532d4"
+					(reference "#PWR0231")
+					(unit 1)
+				)
+			)
+		)
+	)
+	(symbol
 		(lib_id "power:GNDA")
 		(at 58.42 182.88 0)
@@
 			)
 		)
-		(property "Footprint" "Capacitor_SMD:C_0603_1608Metric"
+		(property "Footprint" "Capacitor_SMD:C_0402_1005Metric"
 			(at 186.69 67.31 0)
 			(hide yes)

Commit message: 回路図一部変更，部品ほぼ置いた　寝かせる
Parts:
- removed R207, R208, R209, R210, R211, R212: 10k, Resistor_SMD:R_0603_1608Metric, symbol Device:R
- removed SW201: PowerON, Connector_JST:JST_XH_B2B-XH-A_1x02_P2.50mm_Vertical, symbol Switch:SW_SPST
- removed SW202, SW203, SW204: TL53BF160Q, samacsys:TL53BF160Q, symbol MysymbolLibrary:TL53BF160Q
- added R207, R209: 13.3k, Resistor_SMD:R_0603_1608Metric, symbol Device:R_Small
- added R208, R210, R211: 1k, Resistor_SMD:R_0603_1608Metric, symbol Device:R_Small
- added SW202: SW_Push, samacsys:SKHHLPA010, symbol Switch:SW_Push
- C201, C204: footprint Capacitor_SMD:C_0402_1005Metric -> Capacitor_SMD:C_0603_1608Metric
- U203: footprint Connector_JST:JST_XH_B8B-XH-A_1x08_P2.50mm_Vertical -> Connector_JST:JST_PH_B8B-PH-K_1x08_P2.00mm_Vertical
- renumbered SW205 to SW201
Connections:
- net +3.3V: no longer R206.1
- net AGND: now also R208.1, R210.2; no longer R201.1, R204.2
- net GNDD: now also R206.2, R211.2, SW202.1
- net PB3: now also R211.1, SW202.2
- net at C204.1, R203.1: now also R209.2; no longer C203.2
- net at C201.2, R202.2: now also R207.1; no longer C202.1
- net PA0: now reaches U202.26 (PWR(MFB))
- net PA0: now also R206.1, U204.5 (PA0); no longer R206.2
- net PB4: no longer names the net of U204.27 (PB4)
- net PB5: no longer names the net of U204.28 (PB5)
- net PB6: no longer names the net of U204.29 (PB6)
- net PB7: no longer names the net of U204.30 (PB7)
- net PB8: no longer names the net of U204.31 (PB8)
- new net: C203.2, R209.1, R210.1
- new net: C202.1, R207.2, R208.2
- new net GNDREF: R201.1, R204.2
- no-connect marks 43 -> 47
Other:
- note removed: "タクトスイッチ縦2連"
- note removed: "デジタルイコライザ"
- moved on the sheet: C202, C203, R201, R204, R206

Commit message: 部品配置進行中
Connections:
- net BCK: now also U204.26 (PB3); no longer U204.18 (PA8)
- net DIN: now also U204.28 (PB5); no longer U204.20 (PA10)
- net LRCK: now also U204.25 (PA15); no longer U204.19 (PA9)
- net UART_RX_STM: now also U204.8 (PA3); no longer U204.25 (PA15)
- net UART_TX_STM: now also U204.7 (PA2); no longer U204.24 (PA14)
- net SWDIO: now reaches U204.23 (PA13)
- net PA4_SW: now reaches U204.9 (PA4)
- net PA4_SW: now also R211.1, SW202.2
- net AIL: no longer names the net of U202.12 (AIL)
- net AIR: no longer names the net of U202.11 (AIR)
- removed net PB3: R211.1, SW202.2, U204.26 (PB3)
- net ~{RST}: no longer names the net of U202.43 (~{RST})
- new net SWCLK: U204.24 (PA14)
- no-connect marks 47 -> 48
Other:
- note removed: "これいる？"
- moved on the sheet: R211, SW202
Changed lines of the file:
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@@
 		)
 	)
-	(text "これいる？"
-		(exclude_from_sim no)
-		(at 32.512 77.978 0)
-		(effects
-			(font
-				(size 1.27 1.27)
-			)
-		)
-	)
 	(text "10uF"
 		(exclude_from_sim no)
@@
 	)
 	(junction
-		(at 26.67 152.4)
-		(diameter 0)
-		(color 0 0 0 0)
-	)
-	(junction
 		(at 181.61 49.53)
 		(diameter 0)
@@
 	)
 	(junction
-		(at 22.86 162.56)
+		(at 22.86 165.1)
 		(diameter 0)
 		(color 0 0 0 0)
@@
 	)
 	(junction
+		(at 26.67 154.94)
+		(diameter 0)
+		(color 0 0 0 0)
+	)
+	(junction
 		(at 85.09 161.29)
 		(diameter 0)
@@
 	)
 	(no_connect
-		(at 66.04 147.32)
-	)
-	(no_connect
 		(at 38.1 100.33)
 	)
@@
 	)
 	(no_connect
-		(at 40.64 157.48)
-	)
-	(no_connect
 		(at 40.64 144.78)
 	)
@@
 	)
 	(no_connect
+		(at 38.1 77.47)
+	)
+	(no_connect
 		(at 40.64 154.94)
 	)
@@
 	)
 	(no_connect
-		(at 66.04 142.24)
+		(at 38.1 80.01)
 	)
 	(no_connect
@@
 	)
 	(no_connect
-		(at 66.04 170.18)
-	)
-	(no_connect
 		(at 38.1 69.85)
 	)
@@
 	)
 	(no_connect
+		(at 38.1 29.21)
+	)
+	(no_connect
 		(at 180.34 157.48)
 	)
@@
 	)
 	(no_connect
+		(at 66.04 160.02)
+	)
+	(no_connect
 		(at 38.1 67.31)
 	)
@@
 	)
 	(no_connect
-		(at 83.82 77.47)
+		(at 66.04 162.56)
 	)
 	(no_connect
-		(at 66.04 144.78)
+		(at 83.82 77.47)
 	)
 	(no_connect
@@
 		(at 38.1 34.29)
 	)
+	(no_connect
+		(at 66.04 157.48)
+	)
 	(wire
 		(pts
@@
 	(wire
 		(pts
+			(xy 26.67 154.94) (xy 30.48 154.94)
+		)
+		(stroke
+			(width 0)
+			(type default)
+		)
+	)
+	(wire
+		(pts
 			(xy 144.78 62.23) (xy 146.05 62.23)
 		)
@@
 	(wire
 		(pts
-			(xy 22.86 152.4) (xy 40.64 152.4)
+			(xy 22.86 154.94) (xy 26.67 154.94)
 		)
 		(stroke
@@
 	(wire
 		(pts
-			(xy 26.67 152.4) (xy 26.67 154.94)
+			(xy 26.67 154.94) (xy 26.67 157.48)
 		)
 		(stroke
@@
 	(wire
 		(pts
-			(xy 26.67 162.56) (xy 22.86 162.56)
+			(xy 26.67 165.1) (xy 22.86 165.1)
 		)
 		(stroke
@@
 	(wire
 		(pts
-			(xy 26.67 160.02) (xy 26.67 162.56)
+			(xy 26.67 162.56) (xy 26.67 165.1)
 		)
 		(stroke
@@
 	)
 	(label "UART_RX_STM"
-		(at 66.04 175.26 0)
+		(at 66.04 144.78 0)
 		(effects
 			(font
@@
 		)
 	)
-	(label "PB3"
-		(at 40.64 152.4 180)
-		(effects
-			(font
-				(size 1.27 1.27)
-			)
-			(justify right bottom)
-		)
-	)
 	(label "AVDD"
 		(at 161.29 50.8 270)
@@
 		)
 	)
+	(label "PA4_SW"
+		(at 66.04 147.32 0)
+		(effects
+			(font
+				(size 1.27 1.27)
+			)
+			(justify left bottom)
+		)
+	)
 	(label "PB0"
 		(at 40.64 149.86 180)
@@
 		)
 	)
+	(label "BCK"
+		(at 40.64 152.4 180)
+		(effects
+			(font
+				(size 1.27 1.27)
+			)
+			(justify right bottom)
+		)
+	)
 	(label "SCK"
 		(at 66.04 149.86 0)
@@
 		)
 	)
-	(label "~{RST}"
-		(at 38.1 29.21 180)
-		(effects
-			(font
-				(size 1.27 1.27)
-			)
-			(justify right bottom)
-		)
-	)
 	(label "MOSI"
 		(at 90.17 156.21 180)
@@
 	)
 	(label "DIN"
-		(at 66.04 162.56 0)
+		(at 40.64 157.48 180)
 		(effects
 			(font
 				(size 1.27 1.27)
 			)
-			(justify left bottom)
+			(justify right bottom)
 		)
 	)
@@
 	)
 	(label "UART_TX_STM"
-		(at 66.04 172.72 0)
+		(at 66.04 142.24 0)
 		(effects
 			(font
@@
 		)
 	)
-	(label "AIL"
-		(at 38.1 80.01 180)
-		(effects
-			(font
-				(size 1.27 1.27)
-			)
-			(justify right bottom)
-		)
-	)
 	(label "play{slash}pause"
 		(at 85.09 44.45 0)
@@
 		)
 	)
-	(label "VDDA"
-		(at 99.06 175.26 90)
+	(label "PA4_SW"
+		(at 30.48 154.94 0)
 		(effects
 			(font
@@
 		)
 	)
-	(label "BCK"
-		(at 66.04 157.48 0)
+	(label "VDDA"
+		(at 99.06 175.26 90)
 		(effects
 			(font
@@
 		)
 	)
-	(label "AIR"
-		(at 38.1 77.47 180)
-		(effects
-			(font
-				(size 1.27 1.27)
-			)
-			(justify right bottom)
-		)
-	)
 	(label "LRCK"
-		(at 66.04 160.02 0)
+		(at 66.04 175.26 0)
 		(effects
 			(font
@@
 		)
 	)
+	(hierarchical_label "SWDIO"
+		(shape bidirectional)
+		(at 66.04 170.18 0)
+		(effects
+			(font
+				(size 1.27 1.27)
+			)
+			(justify left)
+		)
+	)
 	(hierarchical_label "DP_BM83"
 		(shape input)
@@
 		)
 	)
+	(hierarchical_label "SWCLK"
+		(shape input)
+		(at 66.04 172.72 0)
+		(effects
+			(font
+				(size 1.27 1.27)
+			)
+			(justify left)
+		)
+	)
 	(hierarchical_label "DM_STM"
 		(shape input)
@@
 	(symbol
 		(lib_id "Switch:SW_Push")
-		(at 22.86 157.48 90)
+		(at 22.86 160.02 90)
 		(unit 1)
 		(body_style 1)
@@
 		(dnp no)
 		(property "Reference" "SW202"
-			(at 19.558 156.21 90)
+			(at 19.558 158.75 90)
 			(show_name no)
 			(do_not_autoplace no)
@@
 		)
 		(property "Value" "SW_Push"
-			(at 19.558 158.75 90)
+			(at 19.558 161.29 90)
 			(show_name no)
 			(do_not_autoplace no)
@@
 		)
 		(property "Footprint" "samacsys:SKHHLPA010"
-			(at 17.78 157.48 0)
+			(at 17.78 160.02 0)
 			(hide yes)
 			(show_name no)
@@
 		)
 		(property "Datasheet" ""
-			(at 17.78 157.48 0)
+			(at 17.78 160.02 0)
 			(hide yes)
 			(show_name no)
@@
 		)
 		(property "Description" "Push button switch, generic, two pins"
-			(at 22.86 157.48 0)
+			(at 22.86 160.02 0)
 			(hide yes)
 			(show_name no)
@@
 	(symbol
 		(lib_id "Device:R_Small")
-		(at 26.67 157.48 0)
+		(at 26.67 160.02 0)
 		(unit 1)
 		(body_style 1)
@@
 		(dnp no)
 		(property "Reference" "R211"
-			(at 27.94 156.21 0)
+			(at 27.94 158.75 0)
 			(show_name no)
 			(do_not_autoplace no)
@@
 		)
 		(property "Value" "1k"
-			(at 27.94 158.75 0)
+			(at 27.94 161.29 0)
 			(show_name no)
 			(do_not_autoplace no)
@@
 		)
 		(property "Footprint" "Resistor_SMD:R_0603_1608Metric"
-			(at 26.67 157.48 0)
+			(at 26.67 160.02 0)
 			(hide yes)
 			(show_name no)
@@
 		)
 		(property "Datasheet" ""
-			(at 26.67 157.48 0)
+			(at 26.67 160.02 0)
 			(hide yes)
 			(show_name no)
@@
 		)
 		(property "Description" "Resistor, small symbol"
-			(at 26.67 157.48 0)
+			(at 26.67 160.02 0)
 			(hide yes)
 			(show_name no)
@@
 	(symbol
 		(lib_id "power:GNDD")
-		(at 22.86 162.56 0)
+		(at 22.86 165.1 0)
 		(unit 1)
 		(body_style 1)
@@
 		(dnp no)
 		(property "Reference" "#PWR0216"
-			(at 22.86 168.91 0)
+			(at 22.86 171.45 0)
 			(hide yes)
 			(show_name no)
@@
 		)
 		(property "Value" "GNDD"
-			(at 22.86 166.116 0)
+			(at 22.86 168.656 0)
 			(show_name no)
 			(do_not_autoplace no)
@@
 		)
 		(property "Footprint" ""
-			(at 22.86 162.56 0)
+			(at 22.86 165.1 0)
 			(hide yes)
 			(show_name no)
@@
 		)
 		(property "Datasheet" ""
-			(at 22.86 162.56 0)
+			(at 22.86 165.1 0)
 			(hide yes)
 			(show_name no)
@@
 		)
 		(property "Description" "Power symbol creates a global label with name \"GNDD\" , digital ground"
-			(at 22.86 162.56 0)
+			(at 22.86 165.1 0)
 			(hide yes)
 			(show_name no)

Commit message: アナログ部分以外ほぼ完成
Connections:
- net GND is gone; now on net GNDD: C216.2, C217.2, C218.2, C219.2
