File: Amplifier.kicad_sch (KiCad schematic)
At the start: 49 parts, among them Q401 TPC6901A, Q402 TPC6901A, Q403 2SA1359, Q404 2SA1359, Q405 2SC3422, Q406 2SC3422, Q407 TPC6901A, Q408 TPC6901A, Q409 TPC6901A, Q410 TPC6901A, Q411 2SA1359, Q412 2SA1359, Q413 2SC3422, Q414 2SC3422, Q415 TPC6901A, Q416 TPC6901A, U401 LME49740NA, U402 LME49740NA

Commit message: 部品配置進行中
Connections:
- net GNDREF: now also U401.5 (+), U402.5 (+); no longer U401.3 (+), U402.3 (+)
- net at R414.1, RV401.5: now also U402.3 (+); no longer U402.5 (+)
- net at R408.1, R412.1: now also U402.2 (-); no longer U402.6 (-)
- net at Q402.3, Q408.1, R408.2: now also U402.1; no longer U402.7
- net at R407.1, R411.1: now also U401.2 (-); no longer U401.6 (-)
- net at R417.2, U401.10 (+): now also U401.7; no longer U401.1
- net at R413.2, R417.1: now also U401.6 (-); no longer U401.2 (-)
- net at Q401.3, Q407.1, R407.2: now also U401.1; no longer U401.7
- net at R413.1, RV401.2: now also U401.3 (+); no longer U401.5 (+)
- net at R414.2, R418.1: now also U402.6 (-); no longer U402.2 (-)
- net at R418.2, U402.10 (+): now also U402.7; no longer U402.1
Other:
- moved on the sheet: U401A, U401B, U402A, U402B
Changed lines of the file:
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@@
 	)
 	(junction
-		(at 92.71 80.01)
-		(diameter 0)
-		(color 0 0 0 0)
-	)
-	(junction
 		(at 163.83 123.19)
 		(diameter 0)
@@
 	)
 	(junction
-		(at 66.04 106.68)
-		(diameter 0)
-		(color 0 0 0 0)
-	)
-	(junction
 		(at 129.54 60.96)
 		(diameter 0)
@@
 	)
 	(junction
-		(at 205.74 80.01)
+		(at 66.04 106.68)
 		(diameter 0)
 		(color 0 0 0 0)
@@
 	)
 	(junction
+		(at 205.74 80.01)
+		(diameter 0)
+		(color 0 0 0 0)
+	)
+	(junction
 		(at 92.71 104.14)
 		(diameter 0)
@@
 		(color 0 0 0 0)
 	)
+	(junction
+		(at 92.71 80.01)
+		(diameter 0)
+		(color 0 0 0 0)
+	)
 	(wire
 		(pts
@@
 	(symbol
 		(lib_id "Device:Opamp_Quad")
-		(at 213.36 80.01 180)
+		(at 240.03 106.68 180)
 		(unit 2)
 		(body_style 1)
@@
 		(dnp no)
 		(property "Reference" "U402"
-			(at 213.36 88.9 0)
+			(at 240.03 115.57 0)
 			(show_name no)
 			(do_not_autoplace no)
@@
 		)
 		(property "Value" "LME49740NA"
-			(at 213.36 86.36 0)
+			(at 240.03 113.03 0)
 			(show_name no)
 			(do_not_autoplace no)
@@
 		)
 		(property "Footprint" "Package_DIP:DIP-14_W7.62mm_Socket"
-			(at 213.36 80.01 0)
+			(at 240.03 106.68 0)
 			(hide yes)
 			(show_name no)
@@
 		)
 		(property "Datasheet" ""
-			(at 213.36 80.01 0)
+			(at 240.03 106.68 0)
 			(hide yes)
 			(show_name no)
@@
 		)
 		(property "Description" "Quad operational amplifier"
-			(at 213.36 80.01 0)
+			(at 240.03 106.68 0)
 			(hide yes)
 			(show_name no)
@@
 		)
 		(property "Sim.Library" "${KICAD9_SYMBOL_DIR}/Simulation_SPICE.sp"
-			(at 213.36 80.01 0)
+			(at 240.03 106.68 0)
 			(hide yes)
 			(show_name no)
@@
 		)
 		(property "Sim.Name" "kicad_builtin_opamp_quad"
-			(at 213.36 80.01 0)
+			(at 240.03 106.68 0)
 			(hide yes)
 			(show_name no)
@@
 		)
 		(property "Sim.Device" "SUBCKT"
-			(at 213.36 80.01 0)
+			(at 240.03 106.68 0)
 			(hide yes)
 			(show_name no)
@@
 		)
 		(property "Sim.Pins" "1=out1 2=in1- 3=in1+ 4=vcc 5=in2+ 6=in2- 7=out2 8=out3 9=in3- 10=in3+ 11=vee 12=in4+ 13=in4- 14=out4"
-			(at 213.36 80.01 0)
+			(at 240.03 106.68 0)
 			(hide yes)
 			(show_name no)
@@
 	(symbol
 		(lib_id "Device:Opamp_Quad")
-		(at 58.42 106.68 0)
+		(at 85.09 80.01 0)
 		(mirror x)
 		(unit 1)
@@
 		(dnp no)
 		(property "Reference" "U401"
-			(at 58.42 115.57 0)
+			(at 85.09 88.9 0)
 			(show_name no)
 			(do_not_autoplace no)
@@
 		)
 		(property "Value" "LME49740NA"
-			(at 58.42 113.03 0)
+			(at 85.09 86.36 0)
 			(show_name no)
 			(do_not_autoplace no)
@@
 		)
 		(property "Footprint" "Package_DIP:DIP-14_W7.62mm_Socket"
-			(at 58.42 106.68 0)
+			(at 85.09 80.01 0)
 			(hide yes)
 			(show_name no)
@@
 		)
 		(property "Datasheet" ""
-			(at 58.42 106.68 0)
+			(at 85.09 80.01 0)
 			(hide yes)
 			(show_name no)
@@
 		)
 		(property "Description" "Quad operational amplifier"
-			(at 58.42 106.68 0)
+			(at 85.09 80.01 0)
 			(hide yes)
 			(show_name no)
@@
 		)
 		(property "Sim.Library" "${KICAD9_SYMBOL_DIR}/Simulation_SPICE.sp"
-			(at 58.42 106.68 0)
+			(at 85.09 80.01 0)
 			(hide yes)
 			(show_name no)
@@
 		)
 		(property "Sim.Name" "kicad_builtin_opamp_quad"
-			(at 58.42 106.68 0)
+			(at 85.09 80.01 0)
 			(hide yes)
 			(show_name no)
@@
 		)
 		(property "Sim.Device" "SUBCKT"
-			(at 58.42 106.68 0)
+			(at 85.09 80.01 0)
 			(hide yes)
 			(show_name no)
@@
 		)
 		(property "Sim.Pins" "1=out1 2=in1- 3=in1+ 4=vcc 5=in2+ 6=in2- 7=out2 8=out3 9=in3- 10=in3+ 11=vee 12=in4+ 13=in4- 14=out4"
-			(at 58.42 106.68 0)
+			(at 85.09 80.01 0)
 			(hide yes)
 			(show_name no)
@@
 	(symbol
 		(lib_id "Device:Opamp_Quad")
-		(at 240.03 106.68 180)
+		(at 213.36 80.01 180)
 		(unit 1)
 		(body_style 1)
@@
 		(dnp no)
 		(property "Reference" "U402"
-			(at 240.03 115.57 0)
+			(at 213.36 88.9 0)
 			(show_name no)
 			(do_not_autoplace no)
@@
 		)
 		(property "Value" "LME49740NA"
-			(at 240.03 113.03 0)
+			(at 213.36 86.36 0)
 			(show_name no)
 			(do_not_autoplace no)
@@
 		)
 		(property "Footprint" "Package_DIP:DIP-14_W7.62mm_Socket"
-			(at 240.03 106.68 0)
+			(at 213.36 80.01 0)
 			(hide yes)
 			(show_name no)
@@
 		)
 		(property "Datasheet" ""
-			(at 240.03 106.68 0)
+			(at 213.36 80.01 0)
 			(hide yes)
 			(show_name no)
@@
 		)
 		(property "Description" "Quad operational amplifier"
-			(at 240.03 106.68 0)
+			(at 213.36 80.01 0)
 			(hide yes)
 			(show_name no)
@@
 		)
 		(property "Sim.Library" "${KICAD9_SYMBOL_DIR}/Simulation_SPICE.sp"
-			(at 240.03 106.68 0)
+			(at 213.36 80.01 0)
 			(hide yes)
 			(show_name no)
@@
 		)
 		(property "Sim.Name" "kicad_builtin_opamp_quad"
-			(at 240.03 106.68 0)
+			(at 213.36 80.01 0)
 			(hide yes)
 			(show_name no)
@@
 		)
 		(property "Sim.Device" "SUBCKT"
-			(at 240.03 106.68 0)
+			(at 213.36 80.01 0)
 			(hide yes)
 			(show_name no)
@@
 		)
 		(property "Sim.Pins" "1=out1 2=in1- 3=in1+ 4=vcc 5=in2+ 6=in2- 7=out2 8=out3 9=in3- 10=in3+ 11=vee 12=in4+ 13=in4- 14=out4"
-			(at 240.03 106.68 0)
+			(at 213.36 80.01 0)
 			(hide yes)
 			(show_name no)
@@
 	(symbol
 		(lib_id "Device:Opamp_Quad")
-		(at 85.09 80.01 0)
+		(at 58.42 106.68 0)
 		(mirror x)
 		(unit 2)
@@
 		(dnp no)
 		(property "Reference" "U401"
-			(at 85.09 88.9 0)
+			(at 58.42 115.57 0)
 			(show_name no)
 			(do_not_autoplace no)
@@
 		)
 		(property "Value" "LME49740NA"
-			(at 85.09 86.36 0)
+			(at 58.42 113.03 0)
 			(show_name no)
 			(do_not_autoplace no)
@@
 		)
 		(property "Footprint" "Package_DIP:DIP-14_W7.62mm_Socket"
-			(at 85.09 80.01 0)
+			(at 58.42 106.68 0)
 			(hide yes)
 			(show_name no)
@@
 		)
 		(property "Datasheet" ""
-			(at 85.09 80.01 0)
+			(at 58.42 106.68 0)
 			(hide yes)
 			(show_name no)
@@
 		)
 		(property "Description" "Quad operational amplifier"
-			(at 85.09 80.01 0)
+			(at 58.42 106.68 0)
 			(hide yes)
 			(show_name no)
@@
 		)
 		(property "Sim.Library" "${KICAD9_SYMBOL_DIR}/Simulation_SPICE.sp"
-			(at 85.09 80.01 0)
+			(at 58.42 106.68 0)
 			(hide yes)
 			(show_name no)
@@
 		)
 		(property "Sim.Name" "kicad_builtin_opamp_quad"
-			(at 85.09 80.01 0)
+			(at 58.42 106.68 0)
 			(hide yes)
 			(show_name no)
@@
 		)
 		(property "Sim.Device" "SUBCKT"
-			(at 85.09 80.01 0)
+			(at 58.42 106.68 0)
 			(hide yes)
 			(show_name no)
@@
 		)
 		(property "Sim.Pins" "1=out1 2=in1- 3=in1+ 4=vcc 5=in2+ 6=in2- 7=out2 8=out3 9=in3- 10=in3+ 11=vee 12=in4+ 13=in4- 14=out4"
-			(at 85.09 80.01 0)
+			(at 58.42 106.68 0)
 			(hide yes)
 			(show_name no)

Commit message: Volumeの種類と位置変えた
Parts:
- RV401: footprint MyLibrary:RV_2C -> samacsys:RK12L12C
Connections:
- net EQ_L: now also RV401.4; no longer RV401.1
- net EQ_R: now also RV401.1; no longer RV401.4
- net at R413.1, U401.3 (+): now also RV401.5; no longer RV401.2
- net at R414.1, U402.3 (+): now also RV401.2; no longer RV401.5
Other:
- note added: "可変抵抗"
- moved on the sheet: RV401A, RV401B
Changed lines of the file:
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@@
 		)
 	)
+	(text "可変抵抗"
+		(exclude_from_sim no)
+		(at 270.002 92.71 0)
+		(effects
+			(font
+				(size 1.27 1.27)
+			)
+			(href "https://akizukidenshi.com/catalog/g/g117473/")
+		)
+	)
 	(text "出力段"
 		(exclude_from_sim no)
@@
 	(symbol
 		(lib_id "MysymbolLibrary:RV_2C")
-		(at 259.08 88.9 0)
-		(mirror y)
+		(at 39.37 88.9 0)
 		(unit 2)
 		(body_style 1)
@@
 		(dnp no)
 		(property "Reference" "RV401"
-			(at 260.35 87.63 0)
+			(at 38.1 87.63 0)
 			(show_name no)
 			(do_not_autoplace no)
@@
 		)
 		(property "Value" "R"
-			(at 260.35 90.17 0)
+			(at 38.1 90.17 0)
 			(show_name no)
 			(do_not_autoplace no)
@@
 			)
 		)
-		(property "Footprint" "MyLibrary:RV_2C"
-			(at 259.08 88.9 0)
+		(property "Footprint" "samacsys:RK12L12C"
+			(at 39.37 88.9 0)
 			(hide yes)
 			(show_name no)
@@
 		)
 		(property "Datasheet" ""
-			(at 259.08 88.9 0)
+			(at 39.37 88.9 0)
 			(hide yes)
 			(show_name no)
@@
 		)
 		(property "Description" ""
-			(at 259.08 88.9 0)
+			(at 39.37 88.9 0)
 			(hide yes)
 			(show_name no)
@@
 	(symbol
 		(lib_id "MysymbolLibrary:RV_2C")
-		(at 39.37 88.9 0)
+		(at 259.08 88.9 0)
+		(mirror y)
 		(unit 1)
 		(body_style 1)
@@
 		(dnp no)
 		(property "Reference" "RV401"
-			(at 38.1 87.63 0)
+			(at 260.35 87.63 0)
 			(show_name no)
 			(do_not_autoplace no)
@@
 		)
 		(property "Value" "R"
-			(at 38.1 90.17 0)
+			(at 260.35 90.17 0)
 			(show_name no)
 			(do_not_autoplace no)
@@
 			)
 		)
-		(property "Footprint" "MyLibrary:RV_2C"
-			(at 39.37 88.9 0)
+		(property "Footprint" "samacsys:RK12L12C"
+			(at 259.08 88.9 0)
 			(hide yes)
 			(show_name no)
@@
 		)
 		(property "Datasheet" ""
-			(at 39.37 88.9 0)
+			(at 259.08 88.9 0)
 			(hide yes)
 			(show_name no)
@@
 		)
 		(property "Description" ""
-			(at 39.37 88.9 0)
+			(at 259.08 88.9 0)
 			(hide yes)
 			(show_name no)
