File: BM83.kicad_pcb (KiCad board)
At the start: 2 copper layers, 202 parts, among them IC101 NJM2845DL1-33, J101 USB_C_Receptacle_USB2.0, J102 Conn_01x02, J103 Jack-DC, J104 3557-2, J105 Conn_01x02, J106 AudioJack3, Q101 2SC1815, Q102 2SA1015, Q401 TPC6901A, Q402 TPC6901A, Q403 PNP, Q404 PNP, Q405 NPN, Q406 NPN, Q407 TPC6901A, Q408 TPC6901A, Q409 TPC6901A, Q410 TPC6901A, Q411 PNP, Q412 PNP, Q413 NPN, Q414 NPN, Q415 TPC6901A, Q416 TPC6901A, SW101 SW_Slide_DPDT, SW102 SW_SPST, SW201 PowerON, SW202 SW_Push, U101 CH221K, U102 USBLC6-2SC6, U103 LM358N, U201 PCM5102A, U202 Microchip_BM83, U203 ST7735S, U204 STM32G431KBTx, U301 TL072, U302 TL074, U303 TL074, U401 ???, U402 ???

Commit message: 何やってたか忘れた
Parts:
- removed C220: 1u, Capacitor_THT:C_Rect_L7.2mm_W6.0mm_P5.00mm
- removed R116: 100k, Resistor_SMD:R_0603_1608Metric
- removed U103: LM358N, Package_DIP:DIP-8_W7.62mm_Socket
- added D109: PESD5V0S1UL, Diode_SMD:D_SOD-882, F.Cu at (60.2, 97.7)
- added D111: D, nittc-footprint-library:CUHS20F30H3F, F.Cu at (144.3, 83.4)
- added D112: D, nittc-footprint-library:CUHS20F30H3F, F.Cu at (137.7, 83.2)
- added K101: G2R-1-E 24V, Relay_THT:Relay_SPDT_Omron_G2RL-1-E, F.Cu at (65.5, 78.3)
- added SW203: TL53BF160Q, samacsys:TL53BF160Q, F.Cu at (149.7, 145.6)
- added SW204: TL53BF160Q, samacsys:TL53BF160Q, F.Cu at (162.7, 145.6)
- added SW205: SW_Push, samacsys:TVAF06A020BR, F.Cu at (346.2, 202.8)
- C104, C105, C106, C107: footprint Capacitor_THT:CP_Radial_D12.5mm_P5.00mm -> Capacitor_THT:CP_Radial_D16.0mm_P7.50mm
- C110: footprint Capacitor_SMD:C_0603_1608Metric -> Capacitor_SMD:C_1206_3216Metric
- C117: value 0.33u -> 1u; footprint Capacitor_SMD:C_0603_1608Metric -> Capacitor_THT:C_Rect_L7.2mm_W6.0mm_P5.00mm
- C118, C203: value 2.2u -> 1u; footprint Capacitor_SMD:C_0603_1608Metric -> Capacitor_THT:C_Rect_L7.2mm_W6.0mm_P5.00mm
- C119: value 1u -> 0.33u; footprint Capacitor_THT:C_Rect_L7.2mm_W6.0mm_P5.00mm -> Capacitor_SMD:C_0603_1608Metric
- C120: value 1u -> 2.2u; footprint Capacitor_THT:C_Rect_L7.2mm_W6.0mm_P5.00mm -> Capacitor_SMD:C_0603_1608Metric
- C202: value 2.2n -> 1u; footprint Capacitor_SMD:C_0603_1608Metric -> Capacitor_THT:C_Rect_L7.2mm_W6.0mm_P5.00mm
- C204: value 0.1u -> 2.2n
- C205, C212: value 10u -> 2.2u; footprint Capacitor_SMD:CP_Elec_3x5.3 -> Capacitor_SMD:C_0603_1608Metric
- C210: value 2.2u -> 0.1u
- C211, C214: value 0.1u -> 10u; footprint Capacitor_SMD:C_0603_1608Metric -> Capacitor_SMD:CP_Elec_3x5.3
- C215: value 0.01u -> 0.1u
- C216: value 4.7u -> 0.1u; footprint Capacitor_SMD:C_0603_1608Metric -> Capacitor_SMD:C_0402_1005Metric
- C217: value 0.1u -> 0.01u; footprint Capacitor_SMD:C_0603_1608Metric -> Capacitor_SMD:C_0402_1005Metric
- C218: value 0.1u -> 4.7u; footprint Capacitor_SMD:C_0603_1608Metric -> Capacitor_SMD:C_0402_1005Metric
- C219: value 1u -> 0.1u; footprint Capacitor_THT:C_Rect_L7.2mm_W6.0mm_P5.00mm -> Capacitor_SMD:C_0402_1005Metric
- D101, D102, D103, D104, D105: footprint LED_THT:LED_D5.0mm_Horizontal_O1.27mm_Z3.0mm -> LED_THT:LED_D3.0mm_Horizontal_O1.27mm_Z2.0mm
- D107: value ? -> SMF24A; footprint Diode_THT:D_DO-35_SOD27_P7.62mm_Horizontal -> Diode_SMD:D_SOD-123F
- D108: value ? -> PESD5V0S1UL; footprint nittc-footprint-library:CUHS20F30H3F -> Diode_SMD:D_SOD-882
- D110: value LED -> ?; footprint LED_THT:LED_D3.0mm_Horizontal_O1.27mm_Z2.0mm -> nittc-footprint-library:CUHS20F30H3F
- FB102: value ? -> 33; footprint Inductor_SMD:L_0603_1608Metric -> Inductor_SMD:L_0805_2012Metric
- J106: footprint MyLibrary:MJ352W -> samacsys:MJ-8435
- JP101, JP102: footprint Connector_PinHeader_2.54mm:PinHeader_1x03_P2.54mm_Vertical -> Jumper:SolderJumper-3_P1.3mm_Open_RoundedPad1.0x1.5mm
- R113: value 2k -> 10k
- R114, R204: value 10k -> 100k
- R201: value 470 -> 100k
- R203: value 10k -> 470
- R205, R206: value 100k -> 10k
- SW202: value SW_Push -> TL53BF160Q; footprint samacsys:TVAF06A020BR -> samacsys:TL53BF160Q
- U102: value USBLC6-2SC6 -> LM358N; footprint Package_TO_SOT_SMD:SOT-23-6 -> Package_DIP:DIP-8_W7.62mm_Socket
- moved U203 246.8 mm to (388.1, 148.1)
- moved C205 240.7 mm to (427.9, 98.3)
- moved C207 240.7 mm to (427.9, 103.2)
- moved C209 240.7 mm to (427.9, 108.0)
- moved C212 240.7 mm to (427.9, 112.9)
- moved LED201 234.4 mm to (428.6, 133.7)
- moved LED202 234.4 mm to (428.6, 140.3)
- moved C301 230.8 mm to (337.0, 141.5)
- moved C302 230.8 mm to (337.0, 144.8)
- moved C303 230.8 mm to (337.0, 148.2)
- moved C304 230.8 mm to (295.1, 144.4)
- moved C305 230.8 mm to (295.1, 111.5)
- moved C306 230.8 mm to (295.1, 115.5)
- moved C307 230.8 mm to (327.3, 143.6)
- moved C308 230.8 mm to (295.1, 119.6)
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Connections:
- net /USB_DM renamed /USB_D-
- net /USB_DP renamed /USB_D+
- C110 pad 2: V- -> AGND
- C111 pad 2: V- -> AGND
- C112 pad 2: V- -> AGND
- C117 pad 1: +5V -> Net-(C117-Pad1)
- C117 pad 2: AGND -> /SIG_L
- C118 pad 1: +3.3V -> /SIG_R
- C118 pad 2: AGND -> Net-(C118-Pad2)
- C119 pad 1: Net-(C119-Pad1) -> +5V
- C119 pad 2: /SIG_L -> AGND
- C120 pad 1: /SIG_R -> +3.3V
- C120 pad 2: Net-(C120-Pad2) -> AGND
- C202 pad 1: Net-(C202-Pad1) -> Net-(C201-Pad2)
- C202 pad 2: AGND -> /SIG_L
- C203 pad 1: Net-(U201-CAPP) -> /SIG_R
- C203 pad 2: Net-(U201-CAPM) -> Net-(C203-Pad2)
- C204 pad 1: +3.3V -> Net-(C203-Pad2)
- C205 pad 1: +3.3V -> Net-(U201-CAPP)
- C205 pad 2: AGND -> Net-(U201-CAPM)
- C206 pad 1: AGND -> +3.3V
- C206 pad 2: /DAC/LDOO -> AGND
- C207 pad 1: /DAC/LDOO -> +3.3V
- C208 pad 1: +3.3VA -> AGND
- C208 pad 2: AGND -> /DAC/LDOO
- C209 pad 1: +3.3VA -> /DAC/LDOO
- C210 pad 1: AGND -> +3.3VA
- C210 pad 2: /DAC/VNEG -> AGND
- C212 pad 1: +3.3VA -> AGND
- C212 pad 2: AGND -> /DAC/VNEG
- C213 pad 1: Net-(U204-PG10) -> +3.3VA
- C214 pad 1: /DAC/VDDA -> +3.3VA
- C214 pad 2: GND -> AGND
- C215 pad 1: /DAC/VDDA -> /DAC/RESET
- C215 pad 2: GND -> AGND
- C216 pad 1: /DAC/VDD1 -> /DAC/VDDA
- C217 pad 1: /DAC/VDD2 -> /DAC/VDDA
- C218 pad 1: /DAC/VDD2 -> /DAC/VDD1
- C219 pad 1: Net-(C201-Pad2) -> /DAC/VDD2
- C219 pad 2: /SIG_L -> GND
- C301 pad 2: V- -> AGND
- C302 pad 2: V- -> AGND
- C303 pad 2: V- -> AGND
- C401 pad 2: V- -> AGND
- C402 pad 2: V- -> AGND
- D108 pad 1: Net-(D108-K) -> /DM
- D110 pad 2: V+ -> AGND
- F101 pad 2: Net-(U102-VBUS) -> Net-(F101-Pad2)
- H101 pad 1: GNDREF -> AGND
- H102 pad 1: GNDREF -> AGND
- H103 pad 1: GNDREF -> AGND
- H104 pad 1: GNDREF -> AGND
- J101 pad A4: Net-(U102-VBUS) -> Net-(F101-Pad2)
- J101 pad A6: Net-(J101-D+-PadA6) -> /DP
- J101 pad A7: Net-(J101-D--PadA7) -> /DM
- J101 pad A9: Net-(U102-VBUS) -> Net-(F101-Pad2)
- J101 pad B4: Net-(U102-VBUS) -> Net-(F101-Pad2)
- J101 pad B6: Net-(J101-D+-PadA6) -> /DP
- J101 pad B7: Net-(J101-D--PadA7) -> /DM
- J101 pad B9: Net-(U102-VBUS) -> Net-(F101-Pad2)
- J106 pad R: Net-(C120-Pad2) -> Net-(C118-Pad2)
- J106 pad T: Net-(C119-Pad1) -> Net-(C117-Pad1)
- Q102 pad 1: V- -> AGND
- Q401 pad 4: V- -> AGND
- Q402 pad 4: V- -> AGND
- Q405 pad 1: V- -> AGND
- Q406 pad 1: V- -> AGND
- Q409 pad 4: V- -> AGND
- Q410 pad 4: V- -> AGND
- Q413 pad 1: V- -> AGND
- Q414 pad 1: V- -> AGND
- R111 pad 2: Net-(U103A-+) -> Net-(U102A-+)
- R113 pad 1: Net-(D110-K) -> Net-(U102A-+)
- R113 pad 2: V- -> AGND
- R114 pad 1: Net-(U103A-+) -> /SIG_L
- R114 pad 2: V- -> GNDREF
- R115 pad 1: /SIG_L -> /SIG_R
- R201 pad 1: Net-(U201-OUTL) -> AGND
- R201 pad 2: Net-(C201-Pad2) -> /SIG_L
- R202 pad 1: Net-(C202-Pad1) -> Net-(U201-OUTL)
- R202 pad 2: Net-(U201-OUTR) -> Net-(C201-Pad2)
- R203 pad 1: +3.3V -> Net-(C203-Pad2)
- R203 pad 2: Net-(U201-XSMT) -> Net-(U201-OUTR)
- R204 pad 1: +3.3V -> /SIG_R
- R204 pad 2: Net-(SW201-B) -> AGND
- R205 pad 1: AGND -> +3.3V
- R205 pad 2: /SIG_L -> Net-(U201-XSMT)
- R206 pad 1: /SIG_R -> +3.3V
- R206 pad 2: AGND -> Net-(SW201-B)
- R208 pad 1: /DAC/PB4 -> /DAC/PB5
- R209 pad 1: /DAC/PB5 -> /DAC/PB7
- R210 pad 1: /DAC/PB6 -> /DAC/PB4
- R211 pad 1: /DAC/PB7 -> /DAC/PB6
- R409 pad 2: V- -> AGND
- R410 pad 2: V- -> AGND
- R427 pad 2: V- -> AGND
- R428 pad 2: V- -> AGND
- SW101 pad 4: /DP_BM83 -> /DP_STM32
- SW101 pad 6: /DP_STM32 -> /DP_BM83
- SW102 pad 2: Net-(D108-K) -> Net-(D110-K)
- SW202 pad 1: AGND -> /DAC/PB3
- SW202 pad 2: Net-(U204-PG10) -> /DAC/PB4
- U102 pad 1: Net-(J101-D--PadA7) -> Net-(R112-Pad1)
- U102 pad 2: AGND -> GNDREF
- U102 pad 3: Net-(J101-D+-PadA6) -> Net-(U102A-+)
- U102 pad 4: /DP -> AGND
- U102 pad 5: Net-(U102-VBUS) -> GNDREF
- U102 pad 6: /DM -> Net-(U102B--)
- U204 pad 4: Net-(U204-PG10) -> /DAC/RESET
- U301 pad 4: V- -> AGND
- U302 pad 4: V- -> AGND
- U303 pad 4: V- -> AGND
- U401 pad 11: V- -> AGND
- U402 pad 11: V- -> AGND
Routing:
- net /DM: track 0.00 -> 14.8 mm
- net /DP: track 0.00 -> 14.5 mm
- net /USB_D+: track 0.00 -> 11.6 mm
- net /USB_D-: track 0.00 -> 11.6 mm
- net Net-(J101-CC2): track 0.00 -> 4.08 mm
- net Net-(J101-CC1): track 0.00 -> 3.45 mm
Other:
- board outline added: 200 x 100 mm
- copper layers 2 -> 6

Commit message: 部品配置すすめた
Parts:
- removed HS401, HS402, HS403, HS404: Heatsink, MyLibrary:17PB024
- added G*** (x3): LOGO, LOGO, F.Cu at (222.8, 167.2)
- C110, C401, C402, R205: moved to B.Cu
- C201, C204, C206, C208, C210, C212, C213: footprint Capacitor_SMD:C_0603_1608Metric -> Capacitor_SMD:C_0402_1005Metric
- C205: footprint Capacitor_SMD:C_0603_1608Metric -> Capacitor_SMD:C_0402_1005Metric; moved to B.Cu
- moved LED201 370.6 mm to (60.0, 172.0), turned to 90 degrees
- moved LED202 363.4 mm to (66.6, 172.0), turned to 90 degrees
- moved C207 352.3 mm to (75.7, 112.3), turned to 90 degrees
- moved C209 352.2 mm to (75.7, 106.6), turned to -90 degrees
- moved C205 344.3 mm to (83.8, 108.7), turned to 90 degrees
- moved C212 341.2 mm to (86.8, 107.7), turned to 90 degrees
- moved U203 328.9 mm to (60.7, 179.9)
- moved SW201 325.6 mm to (64.5, 191.9)
- moved C215 319.8 mm to (40.0, 182.1)
- moved R205 300.9 mm to (81.4, 108.9), turned to 90 degrees
- moved SW205 299.2 mm to (60.8, 113.1), turned to 90 degrees
- moved R206 297.2 mm to (82.8, 187.4)
- moved R203 290.4 mm to (91.8, 105.5), turned to 180 degrees
- moved R202 289.7 mm to (91.8, 107.0)
- moved C208 280.9 mm to (78.1, 108.4), turned to 90 degrees
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Connections:
- C216 pad 1: /DAC/VDDA -> +3.3VA
- C217 pad 1: /DAC/VDDA -> +3.3VA
- C218 pad 1: /DAC/VDD1 -> +3.3V
- C219 pad 1: /DAC/VDD2 -> +3.3V
- U204 pad 1: /DAC/VDD1 -> +3.3V
- U204 pad 15: /DAC/VDDA -> +3.3VA
- U204 pad 17: /DAC/VDD2 -> +3.3V
Routing:
- net Net-(U302A--): track 0.00 -> 9.54 mm
- net Net-(U302B--): track 0.00 -> 9.43 mm
- net Net-(U302C--): track 0.00 -> 9.41 mm
- net Net-(U302A-+): track 0.00 -> 7.35 mm
- net Net-(C304-Pad2): track 0.00 -> 6.94 mm
- net Net-(U201-OUTR): track 0.00 -> 6.00 mm
- net Net-(U201-OUTL): track 0.00 -> 5.85 mm
- net Net-(U302B-+): track 0.00 -> 5.53 mm
- net Net-(U302C-+): track 0.00 -> 5.52 mm
- net Net-(C306-Pad2): track 0.00 -> 4.72 mm
- net Net-(C305-Pad2): track 0.00 -> 4.70 mm
- net Net-(U402D--): track 0.00 -> 2.54 mm
- net Net-(U401D--): track 0.00 -> 2.54 mm
Other:
- board text added: "Volume"

Commit message: 回路図一部変更，部品ほぼ置いた　寝かせる
Parts:
- removed R212: 10k, Resistor_SMD:R_0603_1608Metric
- removed the SW201 at (64.5, 191.9)
- removed SW203, SW204: TL53BF160Q, samacsys:TL53BF160Q
- added C121: 1000u, Capacitor_THT:CP_Radial_D16.0mm_P7.50mm, F.Cu at (135.0, 69.5)
- C201, C204: footprint Capacitor_SMD:C_0402_1005Metric -> Capacitor_SMD:C_0603_1608Metric
- C302, C303, D110, R206: moved to B.Cu
- J102, J105: value Conn_01x02 -> JST_VH
- Q403, Q404, Q411, Q412: value PNP -> 2SA1359
- Q405, Q406, Q413, Q414: value NPN -> 2SC3422
- R207, R209: value 10k -> 13.3k
- R208, R210: value 10k -> 1k
- R211: value 10k -> 1k; moved to B.Cu
- R407, R408, R415, R416: value 10k -> 30k
- SW202: value TL53BF160Q -> SW_Push; footprint samacsys:TL53BF160Q -> samacsys:SKHHLPA010
- U203: footprint Connector_JST:JST_XH_B8B-XH-A_1x08_P2.50mm_Vertical -> Connector_JST:JST_PH_B8B-PH-K_1x08_P2.00mm_Vertical
- U401, U402: value ??? -> LME49740NA
- moved D105 136.2 mm to (86.3, 55.1), turned to 180 degrees
- moved D104 127.3 mm to (81.3, 55.1), turned to 180 degrees
- moved R105 121.0 mm to (85.0, 57.0), turned to 180 degrees
- moved D103 118.3 mm to (76.3, 55.1), turned to 180 degrees
- moved R104 116.6 mm to (80.0, 57.0), turned to 180 degrees
- moved R103 112.2 mm to (75.0, 57.0), turned to 180 degrees
- moved C313 111.4 mm to (92.1, 124.4)
- moved C301 110.9 mm to (89.2, 135.4), turned to -90 degrees
- moved D102 109.4 mm to (71.3, 55.1), turned to 180 degrees
- moved R102 108.1 mm to (70.0, 57.0), turned to 180 degrees
- moved C302 105.0 mm to (103.8, 126.1)
- moved R101 104.0 mm to (65.0, 57.0), turned to 180 degrees
- moved R311 101.3 mm to (93.0, 120.4)
- moved D101 100.5 mm to (66.3, 55.1), turned to 180 degrees
- moved R314 96.8 mm to (96.1, 120.4), turned to 180 degrees
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- renumbered SW205 to SW201
Connections:
- C202 pad 1: Net-(C201-Pad2) -> Net-(C202-Pad1)
- C204 pad 1: Net-(C203-Pad2) -> Net-(C204-Pad1)
- R201 pad 1: AGND -> GNDREF
- R203 pad 1: Net-(C203-Pad2) -> Net-(C204-Pad1)
- R204 pad 2: AGND -> GNDREF
- R206 pad 1: +3.3V -> /DAC/PA0
- R206 pad 2: Net-(SW201-B) -> AGND
- R207 pad 1: /DAC/PB3 -> Net-(C201-Pad2)
- R207 pad 2: AGND -> Net-(C202-Pad1)
- R208 pad 1: /DAC/PB5 -> AGND
- R208 pad 2: AGND -> Net-(C202-Pad1)
- R209 pad 1: /DAC/PB7 -> Net-(C203-Pad2)
- R209 pad 2: AGND -> Net-(C204-Pad1)
- R210 pad 1: /DAC/PB4 -> Net-(C203-Pad2)
- R211 pad 1: /DAC/PB6 -> /DAC/PB3
- SW202 pad 1: /DAC/PB3 -> AGND
- SW202 pad 2: /DAC/PB4 -> /DAC/PB3
- SW202 pad 3: +3.3V -> (no net)
- SW202 pad 4: +3.3V -> (no net)
- U202 pad 26: Net-(SW201-B) -> /DAC/PA0
- U204 pad 27: /DAC/PB4 -> unconnected-(U204-PB4-Pad27)
- U204 pad 28: /DAC/PB5 -> unconnected-(U204-PB5-Pad28)
- U204 pad 29: /DAC/PB6 -> unconnected-(U204-PB6-Pad29)
- U204 pad 30: /DAC/PB7 -> unconnected-(U204-PB7-Pad30)
- U204 pad 31: /DAC/PB8 -> unconnected-(U204-PB8-Pad31)
- U204 pad 5: unconnected-(U204-PA0-Pad5) -> /DAC/PA0
- U302 pad 11: V+ -> AGND
- U302 pad 4: AGND -> V+
- U303 pad 11: V+ -> AGND
- U303 pad 4: AGND -> V+
Other:
- board size 200 x 100 mm -> 150 x 100 mm

Commit message: 部品配置進行中
Parts:
- R206: moved to F.Cu
- R407: renamed from R417; value 10k -> 30k
- R408: renamed from R418; value 10k -> 30k
- R417: renamed from R407; value 30k -> 10k
- R418: renamed from R408; value 30k -> 10k
- moved G*** 73.9 mm to (233.2, 83.8) (x3)
- moved C201 17.8 mm to (79.2, 120.3), turned to -90 degrees
- moved C204 17.5 mm to (83.7, 120.3), turned to 90 degrees
- moved R203 17.0 mm to (82.2, 119.5), turned to 90 degrees
- moved R202 16.7 mm to (80.7, 119.5), turned to -90 degrees
- moved C214 14.4 mm to (84.8, 116.9), turned to 0 degrees
- moved C211 13.4 mm to (77.9, 116.9), turned to 0 degrees
- moved C213 10.2 mm to (82.9, 114.5), turned to 0 degrees
- moved C210 10.1 mm to (77.9, 114.5), turned to 0 degrees
- moved C212 9.69 mm to (79.8, 114.5), turned to 0 degrees
- moved C207 8.92 mm to (75.6, 103.4), turned to 0 degrees
- moved C209 6.46 mm to (81.3, 103.4), turned to 180 degrees
- moved C205 5.55 mm to (79.0, 111.5), turned to 0 degrees
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- renumbered R413 to R411, R414 to R412, R411 to R413, R412 to R414
Connections:
- net /DM_BM83 renamed /BM83_D-
- net /DM_STM32 renamed /STM32_D-
- net /DP_BM83 renamed /BM83_D+
- net /DP_STM32 renamed /STM32_D+
- R211 pad 1: /DAC/PB3 -> /DAC/PA4_SW
- R302 pad 1: Net-(U301A--) -> Net-(U301B--)
- R310 pad 1: Net-(U301B--) -> Net-(U301A--)
- R407 pad 2: Net-(U401C-+) -> Net-(Q401-Pad3)
- R408 pad 2: Net-(U402C-+) -> Net-(Q402-Pad3)
- R411 pad 1: Net-(U401B-+) -> Net-(U401A--)
- R411 pad 2: Net-(U401A--) -> GNDREF
- R412 pad 1: Net-(U402B-+) -> Net-(U402A--)
- R412 pad 2: Net-(U402A--) -> GNDREF
- R413 pad 1: Net-(U401B--) -> Net-(U401A-+)
- R413 pad 2: GNDREF -> Net-(U401B--)
- R414 pad 1: Net-(U402B--) -> Net-(U402A-+)
- R414 pad 2: GNDREF -> Net-(U402B--)
- R417 pad 2: Net-(Q401-Pad3) -> Net-(U401C-+)
- R418 pad 2: Net-(Q402-Pad3) -> Net-(U402C-+)
- RV401 pad 2: Net-(U401B-+) -> Net-(U401A-+)
- RV401 pad 5: Net-(U402B-+) -> Net-(U402A-+)
- SW202 pad 2: /DAC/PB3 -> /DAC/PA4_SW
- U202 pad 11: /DAC/AIR -> unconnected-(U202-AIR-Pad11)
- U202 pad 12: /DAC/AIL -> unconnected-(U202-AIL-Pad12)
- U202 pad 43: /DAC/~{RST} -> unconnected-(U202-~{RST}-Pad43)
- U204 pad 18: /DAC/BCK -> unconnected-(U204-PA8-Pad18)
- U204 pad 19: /DAC/LRCK -> unconnected-(U204-PA9-Pad19)
- U204 pad 20: /DAC/DIN -> unconnected-(U204-PA10-Pad20)
- U204 pad 23: unconnected-(U204-PA13-Pad23) -> /SWDIO
- U204 pad 24: /DAC/UART_TX_STM -> /SWCLK
- U204 pad 25: /DAC/UART_RX_STM -> /DAC/LRCK
- U204 pad 26: /DAC/PB3 -> /DAC/BCK
- U204 pad 28: unconnected-(U204-PB5-Pad28) -> /DAC/DIN
- U204 pad 7: unconnected-(U204-PA2-Pad7) -> /DAC/UART_TX_STM
- U204 pad 8: unconnected-(U204-PA3-Pad8) -> /DAC/UART_RX_STM
- U204 pad 9: unconnected-(U204-PA4-Pad9) -> /DAC/PA4_SW
- U301 pad 3: /SIG_L -> /SIG_R
- U301 pad 5: /SIG_R -> /SIG_L
- U401 pad 1: Net-(U401C-+) -> Net-(Q401-Pad3)
- U401 pad 3: GNDREF -> Net-(U401A-+)
- U401 pad 5: Net-(U401B-+) -> GNDREF
- U401 pad 7: Net-(Q401-Pad3) -> Net-(U401C-+)
- U402 pad 1: Net-(U402C-+) -> Net-(Q402-Pad3)
- U402 pad 3: GNDREF -> Net-(U402A-+)
- U402 pad 5: Net-(U402B-+) -> GNDREF
- U402 pad 7: Net-(Q402-Pad3) -> Net-(U402C-+)
Routing:
- net Net-(U303D-+): track 0.00 -> 73.9 mm
- net /Amplifier/EQ_R: track 0.00 -> 63.2 mm
- net /DAC/DIN: track 0.00 -> 58.1 mm, vias 0 -> 3
- net /DAC/BCK: track 0.00 -> 57.2 mm, vias 0 -> 3
- net Net-(U302D-+): track 0.00 -> 54.4 mm
- net /DAC/LRCK: track 0.00 -> 53.9 mm, vias 0 -> 2
- net Net-(U302D--): track 0.00 -> 48.5 mm
- net Net-(U303D--): track 0.00 -> 48.5 mm
- net +5V: track 0.00 -> 36.3 mm
- net /Amplifier/EQ_L: track 0.00 -> 33.6 mm
- net Net-(C312-Pad1): track 0.00 -> 30.0 mm
- net Net-(Q405-C): track 0.00 -> 24.4 mm
- net Net-(Q414-C): track 0.00 -> 24.4 mm
- net Net-(Q406-C): track 0.00 -> 24.3 mm
- net Net-(Q413-C): track 0.00 -> 24.3 mm
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- added copper zone on F.Cu, net +3.3V
- added copper zone on F.Cu, net +5V
- added copper zone on B.Cu, net /Amplifier/OUT_L+
- added copper zone on F.Cu, net /Amplifier/OUT_L+
- added copper zone on B.Cu, net /Amplifier/OUT_L-
- added copper zone on F.Cu, net /Amplifier/OUT_L-
- added copper zone on B.Cu, net /Amplifier/OUT_R+
- added copper zone on F.Cu, net /Amplifier/OUT_R+
- added copper zone on B.Cu, net /Amplifier/OUT_R-
- added copper zone on F.Cu, net /Amplifier/OUT_R-
- added copper zone on F.Cu, net AGND
- added copper zone on In1.Cu, net AGND
- added copper zone on In2.Cu, net AGND
- added copper zone on In4.Cu, net AGND
- added copper zone on F.Cu, net GNDREF
- added copper zone on F.Cu, net Net-(FB102-Pad1)
- added copper zone on F.Cu, net Net-(K101-COM)
- added copper zone on F.Cu, net Net-(PS101-VIN)
- added copper zone on F.Cu, net Net-(PS102-VIN)
- added copper zone on F.Cu, net Net-(Q401-Pad1)
- added copper zone on F.Cu, net Net-(Q402-Pad1)
- added copper zone on F.Cu, net Net-(Q407-Pad3)
- added copper zone on F.Cu, net Net-(Q408-Pad3)
- added copper zone on F.Cu, net Net-(Q409-Pad1)
- added copper zone on F.Cu, net Net-(Q410-Pad1)
- added copper zone on F.Cu, net Net-(Q415-Pad3)
- added copper zone on F.Cu, net Net-(Q416-Pad3)
- added copper zone on F.Cu, net Net-(U301A--)
- added copper zone on F.Cu, net Net-(U301B--)
- added copper zone on F.Cu, net Net-(U302A--)
- added copper zone on F.Cu, net Net-(U302B--)
- added copper zone on F.Cu, net Net-(U302C--)
- added copper zone on F.Cu, net Net-(U303A--)
- added copper zone on F.Cu, net Net-(U303B--)
- added copper zone on F.Cu, net Net-(U303C--)
- added copper zone on B.Cu, net V+
- added copper zone on F.Cu, net V+
- added copper zone on In2.Cu, net V+
- added copper zone on F.Cu, net VIN
Other:
- board text added: "OLED"

Commit message: アナログ部分以外ほぼ完成
Parts:
- moved LED202 89.6 mm to (54.0, 80.0), turned to 180 degrees
- moved U203 88.3 mm to (98.0, 106.0)
- moved G*** 85.2 mm to (151.7, 58.8) (x3)
- moved LED201 82.4 mm to (54.0, 86.0), turned to 180 degrees
- moved SW102 6.27 mm to (54.5, 73.8)
- moved FB101 2.23 mm to (55.1, 90.0)
- moved R205 0.96 mm to (78.8, 108.1)
- moved C218 0.61 mm to (62.9, 107.0)
- moved R211 0.56 mm to (62.0, 145.9)
- moved C219 0.43 mm to (72.9, 113.5)
Connections:
- C216 pad 2: GND -> AGND
- C217 pad 2: GND -> AGND
- C218 pad 2: GND -> AGND
- C219 pad 2: GND -> AGND
Routing:
- net V+: track 10.4 -> 170.1 mm, vias 21 -> 27
- net +5V: track 36.3 -> 167.7 mm, vias 0 -> 4
- net +3.3V: track 1.80 -> 116.1 mm, vias 0 -> 6
- net AGND: track 2.57 -> 61.5 mm, vias 20 -> 121
- net +3.3VA: track 0.00 -> 51.1 mm, vias 0 -> 13
- net /DAC/PB0: track 0.00 -> 39.9 mm, vias 0 -> 2
- net /DAC/SCK: track 0.00 -> 38.8 mm, vias 0 -> 1
- net /DAC/PA4_SW: track 0.00 -> 36.6 mm, vias 0 -> 1
- net /DAC/MOSI: track 0.00 -> 34.3 mm, vias 0 -> 1
- net /DAC/MISO: track 0.00 -> 31.1 mm, vias 0 -> 1
- net Net-(J101-SHIELD): track 0.00 -> 19.2 mm
- net Net-(Q101-B): track 0.00 -> 16.1 mm, vias 0 -> 1
- net GNDREF: track 0.00 -> 15.3 mm
- net VIN: track 23.8 -> 30.9 mm
- net Net-(LED201-DO): track 0.00 -> 6.02 mm
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- added copper zone on F.Cu, net +3.3VA
- added copper zone on In2.Cu, net +3.3VA

Commit message: Volumeの種類と位置変えた
Parts:
- C109, C112: footprint Capacitor_THT:CP_Radial_D16.0mm_P7.50mm -> Capacitor_THT:CP_Radial_D10.0mm_P5.00mm
- RV401: footprint MyLibrary:RV_2C -> samacsys:RK12L12C
- moved G*** 56.8 mm to (175.8, 7.40) (x3)
- moved RV401 34.3 mm to (145.5, 108.2), turned to 0 degrees
- moved H101 9.70 mm to (186.6, 53.5)
- moved H104 9.70 mm to (186.6, 146.6)
- moved C401 9.40 mm to (151.5, 77.1)
- moved C402 9.40 mm to (151.5, 122.8)
- moved J102 9.40 mm to (184.6, 79.1)
- moved J105 9.40 mm to (184.6, 124.9)
- moved Q403 9.40 mm to (165.4, 57.7)
- moved Q404 9.40 mm to (165.4, 103.4)
- moved Q405 9.40 mm to (165.4, 69.1)
- moved Q406 9.40 mm to (165.4, 114.8)
- moved Q411 9.40 mm to (165.4, 80.5)
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Connections:
- RV401 pad 1: /Amplifier/EQ_L -> /Amplifier/EQ_R
- RV401 pad 2: Net-(U401A-+) -> Net-(U402A-+)
- RV401 pad 4: /Amplifier/EQ_R -> /Amplifier/EQ_L
- RV401 pad 5: Net-(U402A-+) -> Net-(U401A-+)
Routing:
- net /Amplifier/EQ_R: track 63.2 -> 0.00 mm
- net /Amplifier/EQ_L: track 33.6 -> 0.00 mm
Other:
- board size 150 x 100 mm -> 140 x 100 mm
- board text removed: "Volume"
